File: Daughter_Card/Daughter_Card.kicad_sch (KiCad schematic)
At the start: 107 parts, among them J1 Conn_01x01_Pin, J10 Conn_01x01_Pin, J100 Conn_01x01_Pin, J101 Conn_01x01_Pin, J102 Conn_01x01_Pin, J103 Conn_01x01_Pin, J104 Conn_01x01_Pin, J105 Conn_01x01_Pin, J106 Conn_01x01_Pin, J107 Conn_01x01_Pin, J108 Conn_01x01_Pin, J109 Conn_01x01_Pin, J11 Conn_01x01_Pin, J110 Conn_01x01_Pin, J111 Conn_01x01_Pin, J112 Conn_01x01_Pin, J113 Conn_01x01_Pin, J114 Conn_01x01_Pin, J115 Conn_01x01_Pin, J116 Conn_01x01_Pin, J117 Conn_01x01_Pin, J118 Conn_01x01_Pin, J119 Conn_01x01_Pin, J12 Conn_01x01_Pin, J120 Conn_01x01_Pin, J121 Conn_01x01_Pin, J122 Conn_01x01_Pin, J13 Conn_01x01_Pin, J14 Conn_01x01_Pin, J15 Conn_01x01_Pin, J16 Conn_01x01_Pin, J17 Conn_01x01_Pin, J18 Conn_01x01_Pin, J19 Conn_01x01_Pin, J2 Conn_01x01_Pin, J20 Conn_01x01_Pin, J21 Conn_01x01_Pin, J22 Conn_01x01_Pin, J23 Conn_01x01_Pin, J24 Conn_01x01_Pin, J25 Conn_01x01_Pin, J26 Conn_01x01_Pin, J27 Conn_01x01_Pin, J28 Conn_01x01_Pin, J29 Conn_01x01_Pin, J3 Conn_01x01_Pin, J30 Conn_01x01_Pin, J31 Conn_01x01_Pin, J32 Conn_01x01_Pin, J33 Conn_01x01_Pin, J34 Conn_01x01_Pin, J35 Conn_01x01_Pin, J36 Conn_01x01_Pin, J37 Conn_01x01_Pin, J38 Conn_01x01_Pin, J39 Conn_01x01_Pin, J4 Conn_01x01_Pin, J40 Conn_01x01_Pin, J41 Conn_01x01_Pin, J42 Conn_01x01_Pin, J43 Conn_01x01_Pin, J44 Conn_01x01_Pin, J45 Conn_01x01_Pin, J46 Conn_01x01_Pin, J47 Conn_01x01_Pin, J48 Conn_01x01_Pin, J49 Conn_01x01_Pin, J5 Conn_01x01_Pin, J50 Conn_01x01_Pin, J51 Conn_01x01_Pin, J52 Conn_01x01_Pin, J53 Conn_01x01_Pin, J54 Conn_01x01_Pin, J55 Conn_01x01_Pin, J56 Conn_01x01_Pin, J57 Conn_01x01_Pin, J58 Conn_01x01_Pin, J59 Conn_01x01_Pin, J6 Conn_01x01_Pin, J60 Conn_01x01_Pin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

Commit message: update in 0912
Parts:
- removed C7: 0.1u, Capacitor_SMD:C_0603_1608Metric, symbol Symbols-Library:C_Small
- removed D1: LED_OR, MOSBius_V2_CHIP:LED_150120RS75000_WRE, symbol Symbols-Library:LED
- removed D3: LED_Y, MOSBius_V2_CHIP:LED_150120RS75000_WRE, symbol Symbols-Library:LED
- removed R1, R19, R7: 330, Resistor_SMD:R_0603_1608Metric, symbol Symbols-Library:R_1206
- added C1: 0.1u, Capacitor_SMD:C_0603_1608Metric, symbol Symbols-Library:C_Small
- added R4: 330, Resistor_SMD:R_0603_1608Metric, symbol Symbols-Library:R_1206
- D2: value LED_G -> LED_GRE
- Daughter_Card_PIN1: footprint Connector_PCBEdge:SODIMM-200_1.8V_Card_edge -> MOSBius_V2_CHIP:SODIMM-200_1.8V_Card_edge_Extend
- renumbered J8 to P10, J122 to P100, J9 to P11, J10 to P12, J11 to P14, J12 to P15, J13 to P16, J14 to P17, J15 to P18, J16 to P19, J17 to P20, J18 to P21, J19 to P22, J20 to P23, J21 to P24, J22 to P25, J24 to P26, J23 to P27, J25 to P28, J26 to P29, J2 to P3, J27 to P30, J28 to P31, J29 to P32, J30 to P33, J31 to P34, J32 to P35, J33 to P36, J34 to P37, J35 to P38, J36 to P39, J3 to P4, J37 to P40, J38 to P41, J39 to P42, J40 to P43, J41 to P44, J42 to P45, J43 to P46, J44 to P47, J45 to P48, J46 to P49, J1 to P5, J47 to P50, J48 to P51, J49 to P52, J50 to P53, J51 to P54, J52 to P55, J53 to P56, J54 to P57, J55 to P58, J56 to P59, J4 to P6, J57 to P60, J58 to P61, J59 to P62, J60 to P63, J61 to P64, J62 to P65, J63 to P66, J64 to P67, J65 to P68, J66 to P69, J5 to P7, J67 to P70, J68 to P71, J69 to P72, J70 to P73, J71 to P74, J72 to P75, J73 to P76, J99 to P77, J100 to P78, J101 to P79, J6 to P8, J102 to P80, J103 to P81, J104 to P82, J105 to P83, J106 to P84, J107 to P85, J108 to P86, J109 to P87, J110 to P88, J111 to P89, J7 to P9, J112 to P90, J113 to P91, J114 to P92, J115 to P93, J116 to P94, J117 to P95, J118 to P96, J119 to P97, J120 to P98, J121 to P99
Connections:
- net CC_N_D_CC: now also Daughter_Card_PIN1.168; no longer Daughter_Card_PIN1.118
- net CC_N_D_CS: now also Daughter_Card_PIN1.166; no longer Daughter_Card_PIN1.116
- net CC_N_G_CC: now also Daughter_Card_PIN1.172; no longer Daughter_Card_PIN1.122
- net CC_N_G_CS: now also Daughter_Card_PIN1.170; no longer Daughter_Card_PIN1.120
- net CC_P_D_CC: now also Daughter_Card_PIN1.174; no longer Daughter_Card_PIN1.124
- net CC_P_D_CS: now also Daughter_Card_PIN1.176; no longer Daughter_Card_PIN1.126
- net CC_P_G_CC: now also Daughter_Card_PIN1.178; no longer Daughter_Card_PIN1.128
- net CC_P_G_CS: now also Daughter_Card_PIN1.180; no longer Daughter_Card_PIN1.130
- net CLK: now also Daughter_Card_PIN1.5; no longer Daughter_Card_PIN1.55
- net DATA_SBUS6: now also Daughter_Card_PIN1.7; no longer Daughter_Card_PIN1.57
- net DCC1_N_D_L_CC: now also Daughter_Card_PIN1.189; no longer Daughter_Card_PIN1.139
- net DCC1_N_D_L_CS: now also Daughter_Card_PIN1.191; no longer Daughter_Card_PIN1.141
- net DCC1_N_D_R_CC: now also Daughter_Card_PIN1.193; no longer Daughter_Card_PIN1.143
- net DCC1_N_D_R_CS: now also Daughter_Card_PIN1.195; no longer Daughter_Card_PIN1.145
- net DCC1_N_G_L_CC: now also Daughter_Card_PIN1.181; no longer Daughter_Card_PIN1.131
- net DCC1_N_G_L_CS: now also Daughter_Card_PIN1.183; no longer Daughter_Card_PIN1.133
- net DCC1_N_G_R_CC: now also Daughter_Card_PIN1.185; no longer Daughter_Card_PIN1.135
- net DCC1_N_G_R_CS: now also Daughter_Card_PIN1.187; no longer Daughter_Card_PIN1.137
- net DCC1_P_D_L_CC: now also Daughter_Card_PIN1.22; no longer Daughter_Card_PIN1.72
- net DCC1_P_D_L_CS: now also Daughter_Card_PIN1.24; no longer Daughter_Card_PIN1.74
- net DCC1_P_D_R_CC: now also Daughter_Card_PIN1.18; no longer Daughter_Card_PIN1.68
- net DCC1_P_D_R_CS: now also Daughter_Card_PIN1.20; no longer Daughter_Card_PIN1.70
- net DCC1_P_G_L_CC: now also Daughter_Card_PIN1.30; no longer Daughter_Card_PIN1.80
- net DCC1_P_G_L_CS: now also Daughter_Card_PIN1.32; no longer Daughter_Card_PIN1.82
- net DCC1_P_G_R_CC: now also Daughter_Card_PIN1.26; no longer Daughter_Card_PIN1.76
- net DCC1_P_G_R_CS: now also Daughter_Card_PIN1.28; no longer Daughter_Card_PIN1.78
- net DCC2_N_D_L_CC: now also Daughter_Card_PIN1.173; no longer Daughter_Card_PIN1.123
- net DCC2_N_D_L_CS: now also Daughter_Card_PIN1.175; no longer Daughter_Card_PIN1.125
- net DCC2_N_D_R_CC: now also Daughter_Card_PIN1.177; no longer Daughter_Card_PIN1.127
- net DCC2_N_D_R_CS: now also Daughter_Card_PIN1.179; no longer Daughter_Card_PIN1.129
- net DCC2_N_G_L_CC: now also Daughter_Card_PIN1.165; no longer Daughter_Card_PIN1.115
- net DCC2_N_G_L_CS: now also Daughter_Card_PIN1.167; no longer Daughter_Card_PIN1.117
- net DCC2_N_G_R_CC: now also Daughter_Card_PIN1.169; no longer Daughter_Card_PIN1.119
- net DCC2_N_G_R_CS: now also Daughter_Card_PIN1.171; no longer Daughter_Card_PIN1.121
- net DCC2_P_D_L_CC: now also Daughter_Card_PIN1.38; no longer Daughter_Card_PIN1.88
- net DCC2_P_D_L_CS: now also Daughter_Card_PIN1.40; no longer Daughter_Card_PIN1.90
- net DCC2_P_D_R_CC: now also Daughter_Card_PIN1.34; no longer Daughter_Card_PIN1.84
- net DCC2_P_D_R_CS: now also Daughter_Card_PIN1.36; no longer Daughter_Card_PIN1.86
- net DCC2_P_G_L_CC: now also Daughter_Card_PIN1.46; no longer Daughter_Card_PIN1.96
- net DCC2_P_G_L_CS: now also Daughter_Card_PIN1.48; no longer Daughter_Card_PIN1.98
- net DCC2_P_G_R_CC: now also Daughter_Card_PIN1.42; no longer Daughter_Card_PIN1.92
- net DCC2_P_G_R_CS: now also Daughter_Card_PIN1.44; no longer Daughter_Card_PIN1.94
- net DCC3_N_D_L_CC: now also Daughter_Card_PIN1.41; no longer Daughter_Card_PIN1.91
- net DCC3_N_D_L_CS: now also Daughter_Card_PIN1.43; no longer Daughter_Card_PIN1.93
- net DCC3_N_D_R_CC: now also Daughter_Card_PIN1.45; no longer Daughter_Card_PIN1.95
- net DCC3_N_D_R_CS: now also Daughter_Card_PIN1.47; no longer Daughter_Card_PIN1.97
- net DCC3_N_G_L_CC: now also Daughter_Card_PIN1.33; no longer Daughter_Card_PIN1.83
- net DCC3_N_G_L_CS: now also Daughter_Card_PIN1.35; no longer Daughter_Card_PIN1.85
- net DCC3_N_G_R_CC: now also Daughter_Card_PIN1.37; no longer Daughter_Card_PIN1.87
- net DCC3_N_G_R_CS: now also Daughter_Card_PIN1.39; no longer Daughter_Card_PIN1.89
- net DCC3_P_D_L_CC: now also Daughter_Card_PIN1.154; no longer Daughter_Card_PIN1.104
- net DCC3_P_D_L_CS: now also Daughter_Card_PIN1.156; no longer Daughter_Card_PIN1.106
- net DCC3_P_D_R_CC: now also Daughter_Card_PIN1.50; no longer Daughter_Card_PIN1.100
- net DCC3_P_D_R_CS: now also Daughter_Card_PIN1.152; no longer Daughter_Card_PIN1.102
- net DCC3_P_G_L_CC: now also Daughter_Card_PIN1.162; no longer Daughter_Card_PIN1.112
- net DCC3_P_G_L_CS: now also Daughter_Card_PIN1.164; no longer Daughter_Card_PIN1.114
- net DCC3_P_G_R_CC: now also Daughter_Card_PIN1.158; no longer Daughter_Card_PIN1.108
- net DCC3_P_G_R_CS: now also Daughter_Card_PIN1.160; no longer Daughter_Card_PIN1.110
- net DCC4_N_D_L_CC: now also Daughter_Card_PIN1.57; no longer Daughter_Card_PIN1.107
- net DCC4_N_D_L_CS: now also Daughter_Card_PIN1.59; no longer Daughter_Card_PIN1.109
- net DCC4_N_D_R_CC: now also Daughter_Card_PIN1.161; no longer Daughter_Card_PIN1.111
- net DCC4_N_D_R_CS: now also Daughter_Card_PIN1.163; no longer Daughter_Card_PIN1.113
- net DCC4_N_G_L_CC: now also Daughter_Card_PIN1.49; no longer Daughter_Card_PIN1.99
- net DCC4_N_G_L_CS: now also Daughter_Card_PIN1.51; no longer Daughter_Card_PIN1.101
- net DCC4_N_G_R_CC: now also Daughter_Card_PIN1.53; no longer Daughter_Card_PIN1.103
- net DCC4_N_G_R_CS: now also Daughter_Card_PIN1.55; no longer Daughter_Card_PIN1.105
- net DCC4_P_D_L_CC: now also Daughter_Card_PIN1.6; no longer Daughter_Card_PIN1.56
- net DCC4_P_D_L_CS: now also Daughter_Card_PIN1.8; no longer Daughter_Card_PIN1.58
- net DCC4_P_D_R_CC: now also Daughter_Card_PIN1.2; no longer Daughter_Card_PIN1.52
- net DCC4_P_D_R_CS: now also Daughter_Card_PIN1.4; no longer Daughter_Card_PIN1.54
- net DCC4_P_G_L_CC: now also Daughter_Card_PIN1.14; no longer Daughter_Card_PIN1.64
- net DCC4_P_G_L_CS: now also Daughter_Card_PIN1.16; no longer Daughter_Card_PIN1.66
- net DCC4_P_G_R_CC: now also Daughter_Card_PIN1.10; no longer Daughter_Card_PIN1.60
- net DCC4_P_G_R_CS: now also Daughter_Card_PIN1.12; no longer Daughter_Card_PIN1.62
- net DINV1_INN_L: now also Daughter_Card_PIN1.190; no longer Daughter_Card_PIN1.140
- net DINV1_INN_R: now also Daughter_Card_PIN1.184; no longer Daughter_Card_PIN1.134
- net DINV1_INP_L: now also Daughter_Card_PIN1.192; no longer Daughter_Card_PIN1.142
- net DINV1_INP_R: now also Daughter_Card_PIN1.186; no longer Daughter_Card_PIN1.136
- net DINV1_OUT_L: now also Daughter_Card_PIN1.188; no longer Daughter_Card_PIN1.138
- net DINV1_OUT_R: now also Daughter_Card_PIN1.182; no longer Daughter_Card_PIN1.132
- net DINV2_INN_L: now also Daughter_Card_PIN1.199; no longer Daughter_Card_PIN1.149
- net DINV2_INN_R: now also Daughter_Card_PIN1.196; no longer Daughter_Card_PIN1.146
- net DINV2_INP_L: now also Daughter_Card_PIN1.197; no longer Daughter_Card_PIN1.147
- net DINV2_INP_R: now also Daughter_Card_PIN1.198; no longer Daughter_Card_PIN1.148
- net DINV2_OUT_L: now also Daughter_Card_PIN1.200; no longer Daughter_Card_PIN1.150
- net DINV2_OUT_R: now also Daughter_Card_PIN1.194; no longer Daughter_Card_PIN1.144
- net EN: now also Daughter_Card_PIN1.3; no longer Daughter_Card_PIN1.53
- net GND: now also Daughter_Card_PIN1.100, Daughter_Card_PIN1.101, Daughter_Card_PIN1.102, Daughter_Card_PIN1.103, Daughter_Card_PIN1.104, Daughter_Card_PIN1.105, Daughter_Card_PIN1.106, Daughter_Card_PIN1.107, Daughter_Card_PIN1.108, Daughter_Card_PIN1.109, Daughter_Card_PIN1.110, Daughter_Card_PIN1.111, Daughter_Card_PIN1.112, Daughter_Card_PIN1.113, Daughter_Card_PIN1.114, Daughter_Card_PIN1.115, Daughter_Card_PIN1.116, Daughter_Card_PIN1.117, Daughter_Card_PIN1.118, Daughter_Card_PIN1.119, Daughter_Card_PIN1.120, Daughter_Card_PIN1.121, Daughter_Card_PIN1.122, Daughter_Card_PIN1.123, Daughter_Card_PIN1.124, Daughter_Card_PIN1.125, Daughter_Card_PIN1.126, Daughter_Card_PIN1.127, Daughter_Card_PIN1.128, Daughter_Card_PIN1.129, Daughter_Card_PIN1.130, Daughter_Card_PIN1.131, Daughter_Card_PIN1.132, Daughter_Card_PIN1.133, Daughter_Card_PIN1.134, Daughter_Card_PIN1.135, Daughter_Card_PIN1.136, Daughter_Card_PIN1.137, Daughter_Card_PIN1.138, Daughter_Card_PIN1.139, Daughter_Card_PIN1.140, Daughter_Card_PIN1.141, Daughter_Card_PIN1.142, Daughter_Card_PIN1.143, Daughter_Card_PIN1.144, Daughter_Card_PIN1.145, Daughter_Card_PIN1.146, Daughter_Card_PIN1.147, Daughter_Card_PIN1.148, Daughter_Card_PIN1.149, Daughter_Card_PIN1.150, Daughter_Card_PIN1.52, Daughter_Card_PIN1.54, Daughter_Card_PIN1.56, Daughter_Card_PIN1.58, Daughter_Card_PIN1.60, Daughter_Card_PIN1.61, Daughter_Card_PIN1.62, Daughter_Card_PIN1.63, Daughter_Card_PIN1.64, Daughter_Card_PIN1.65, Daughter_Card_PIN1.66, Daughter_Card_PIN1.67, Daughter_Card_PIN1.68, Daughter_Card_PIN1.69, Daughter_Card_PIN1.70, Daughter_Card_PIN1.71, Daughter_Card_PIN1.72, Daughter_Card_PIN1.73, Daughter_Card_PIN1.74, Daughter_Card_PIN1.75, Daughter_Card_PIN1.76, Daughter_Card_PIN1.77, Daughter_Card_PIN1.78, Daughter_Card_PIN1.79, Daughter_Card_PIN1.80, Daughter_Card_PIN1.81, Daughter_Card_PIN1.82, Daughter_Card_PIN1.83, Daughter_Card_PIN1.84, Daughter_Card_PIN1.85, Daughter_Card_PIN1.86, Daughter_Card_PIN1.87, Daughter_Card_PIN1.88, Daughter_Card_PIN1.89, Daughter_Card_PIN1.90, Daughter_Card_PIN1.91, Daughter_Card_PIN1.92, Daughter_Card_PIN1.93, Daughter_Card_PIN1.94, Daughter_Card_PIN1.95, Daughter_Card_PIN1.96, Daughter_Card_PIN1.97, Daughter_Card_PIN1.98, Daughter_Card_PIN1.99, C1.2; no longer Daughter_Card_PIN1.10, Daughter_Card_PIN1.11, Daughter_Card_PIN1.12, Daughter_Card_PIN1.13, Daughter_Card_PIN1.14, Daughter_Card_PIN1.15, Daughter_Card_PIN1.152, Daughter_Card_PIN1.154, Daughter_Card_PIN1.156, Daughter_Card_PIN1.158, Daughter_Card_PIN1.16, Daughter_Card_PIN1.160, Daughter_Card_PIN1.161, Daughter_Card_PIN1.162, Daughter_Card_PIN1.163, Daughter_Card_PIN1.164, Daughter_Card_PIN1.165, Daughter_Card_PIN1.166, Daughter_Card_PIN1.167, Daughter_Card_PIN1.168, Daughter_Card_PIN1.169, Daughter_Card_PIN1.17, Daughter_Card_PIN1.170, Daughter_Card_PIN1.171, Daughter_Card_PIN1.172, Daughter_Card_PIN1.173, Daughter_Card_PIN1.174, Daughter_Card_PIN1.175, Daughter_Card_PIN1.176, Daughter_Card_PIN1.177, Daughter_Card_PIN1.178, Daughter_Card_PIN1.179, Daughter_Card_PIN1.18, Daughter_Card_PIN1.180, Daughter_Card_PIN1.181, Daughter_Card_PIN1.182, Daughter_Card_PIN1.183, Daughter_Card_PIN1.184, Daughter_Card_PIN1.185, Daughter_Card_PIN1.186, Daughter_Card_PIN1.187, Daughter_Card_PIN1.188, Daughter_Card_PIN1.189, Daughter_Card_PIN1.19, Daughter_Card_PIN1.190, Daughter_Card_PIN1.191, Daughter_Card_PIN1.192, Daughter_Card_PIN1.193, Daughter_Card_PIN1.194, Daughter_Card_PIN1.195, Daughter_Card_PIN1.196, Daughter_Card_PIN1.197, Daughter_Card_PIN1.198, Daughter_Card_PIN1.199, Daughter_Card_PIN1.2, Daughter_Card_PIN1.20, Daughter_Card_PIN1.200, Daughter_Card_PIN1.21, Daughter_Card_PIN1.22, Daughter_Card_PIN1.23, Daughter_Card_PIN1.24, Daughter_Card_PIN1.25, Daughter_Card_PIN1.26, Daughter_Card_PIN1.27, Daughter_Card_PIN1.28, Daughter_Card_PIN1.29, Daughter_Card_PIN1.3, Daughter_Card_PIN1.30, Daughter_Card_PIN1.31, Daughter_Card_PIN1.32, Daughter_Card_PIN1.33, Daughter_Card_PIN1.34, Daughter_Card_PIN1.35, Daughter_Card_PIN1.36, Daughter_Card_PIN1.37, Daughter_Card_PIN1.38, Daughter_Card_PIN1.39, Daughter_Card_PIN1.4, Daughter_Card_PIN1.40, Daughter_Card_PIN1.41, Daughter_Card_PIN1.42, Daughter_Card_PIN1.43, Daughter_Card_PIN1.44, Daughter_Card_PIN1.45, Daughter_Card_PIN1.46, Daughter_Card_PIN1.47, Daughter_Card_PIN1.48, Daughter_Card_PIN1.49, Daughter_Card_PIN1.5, Daughter_Card_PIN1.50, Daughter_Card_PIN1.51, Daughter_Card_PIN1.6, Daughter_Card_PIN1.7, Daughter_Card_PIN1.8, Daughter_Card_PIN1.9
- net OTA_N_INN: now also Daughter_Card_PIN1.29; no longer Daughter_Card_PIN1.79
- net OTA_N_INP: now also Daughter_Card_PIN1.27; no longer Daughter_Card_PIN1.77
- net OTA_N_OUT: now also Daughter_Card_PIN1.31; no longer Daughter_Card_PIN1.81
- net OTA_P_INN: now also Daughter_Card_PIN1.19; no longer Daughter_Card_PIN1.69
- net OTA_P_INP: now also Daughter_Card_PIN1.21; no longer Daughter_Card_PIN1.71
- net OTA_P_OUT: now also Daughter_Card_PIN1.23; no longer Daughter_Card_PIN1.73
- net SBUS1: now also Daughter_Card_PIN1.17; no longer Daughter_Card_PIN1.67
- net SBUS2: now also Daughter_Card_PIN1.15; no longer Daughter_Card_PIN1.65
- net SBUS3: now also Daughter_Card_PIN1.13; no longer Daughter_Card_PIN1.63
- net SBUS4: now also Daughter_Card_PIN1.11; no longer Daughter_Card_PIN1.61
- net SBUS5: now also Daughter_Card_PIN1.9; no longer Daughter_Card_PIN1.59
- net VDD: now also Daughter_Card_PIN1.25, C1.1, R4.1; no longer Daughter_Card_PIN1.75
- net at D2.2 (A): now also R4.2
- no-connect marks 1 -> 0
Other:
- note removed: "Daughter Card Pin Indicators"
- note removed: "The reason putting pins in middle is for easier connection in mother board (socket)"
- company: (none) -> Columbia University
- title: (none) -> MOSbius V2 Darughter Card PCB
