File: Daughter_Card/Daughter_Card.kicad_pcb (KiCad board)
At the start: 2 copper layers, 67.6 x 25.4 mm, 10 parts

Commit message: update in 0912
Parts:
- removed C7: 0.1u, Capacitor_SMD:C_0603_1608Metric
- removed D1: LED_OR, MOSBius_V2_CHIP:LED_150120RS75000_WRE
- removed D3: LED_Y, MOSBius_V2_CHIP:LED_150120RS75000_WRE
- removed R19, R7: 330, Resistor_SMD:R_0603_1608Metric
- removed R8: 750, Resistor_SMD:R_0603_1608Metric
- added ?: , , F.Cu at (73.3, 52.1)
- added ?: , , F.Cu at (134.0, 53.4)
- added C1: 0.1u, Capacitor_SMD:C_0603_1608Metric, F.Cu at (102.8, 37.8)
- added P10: Conn_01x01_Pin, Connector_PinHeader_1.00mm:PinHeader_1x01_P1.00mm_Vertical, F.Cu at (81.0, 55.4)
- added P100: Conn_01x01_Pin, Connector_PinHeader_1.00mm:PinHeader_1x01_P1.00mm_Vertical, F.Cu at (74.2, 46.9)
- added P11: Conn_01x01_Pin, Connector_PinHeader_1.00mm:PinHeader_1x01_P1.00mm_Vertical, F.Cu at (83.3, 58.1)
- added P12: Conn_01x01_Pin, Connector_PinHeader_1.00mm:PinHeader_1x01_P1.00mm_Vertical, F.Cu at (83.3, 55.4)
- added P14: Conn_01x01_Pin, Connector_PinHeader_1.00mm:PinHeader_1x01_P1.00mm_Vertical, F.Cu at (85.6, 58.2)
- added P15: Conn_01x01_Pin, Connector_PinHeader_1.00mm:PinHeader_1x01_P1.00mm_Vertical, F.Cu at (85.6, 55.4)
- added P16: Conn_01x01_Pin, Connector_PinHeader_1.00mm:PinHeader_1x01_P1.00mm_Vertical, F.Cu at (87.9, 59.4)
- added P17: Conn_01x01_Pin, Connector_PinHeader_1.00mm:PinHeader_1x01_P1.00mm_Vertical, F.Cu at (87.9, 56.4)
- added P18: Conn_01x01_Pin, Connector_PinHeader_1.00mm:PinHeader_1x01_P1.00mm_Vertical, F.Cu at (90.2, 59.4)
- added P19: Conn_01x01_Pin, Connector_PinHeader_1.00mm:PinHeader_1x01_P1.00mm_Vertical, F.Cu at (90.2, 56.4)
- added P20: Conn_01x01_Pin, Connector_PinHeader_1.00mm:PinHeader_1x01_P1.00mm_Vertical, F.Cu at (92.5, 60.1)
- added P21: Conn_01x01_Pin, Connector_PinHeader_1.00mm:PinHeader_1x01_P1.00mm_Vertical, F.Cu at (92.5, 57.4)
- added P22: Conn_01x01_Pin, Connector_PinHeader_1.00mm:PinHeader_1x01_P1.00mm_Vertical, F.Cu at (94.8, 60.1)
- added P23: Conn_01x01_Pin, Connector_PinHeader_1.00mm:PinHeader_1x01_P1.00mm_Vertical, F.Cu at (94.8, 57.6)
- added P24: Conn_01x01_Pin, Connector_PinHeader_1.00mm:PinHeader_1x01_P1.00mm_Vertical, F.Cu at (97.1, 60.8)
- added P25: Conn_01x01_Pin, Connector_PinHeader_1.00mm:PinHeader_1x01_P1.00mm_Vertical, F.Cu at (97.1, 58.3)
- added P26: Conn_01x01_Pin, Connector_PinHeader_1.00mm:PinHeader_1x01_P1.00mm_Vertical, F.Cu at (99.4, 60.8)
- added P27: Conn_01x01_Pin, Connector_PinHeader_1.00mm:PinHeader_1x01_P1.00mm_Vertical, F.Cu at (101.7, 60.8)
- added P28: Conn_01x01_Pin, Connector_PinHeader_1.00mm:PinHeader_1x01_P1.00mm_Vertical, F.Cu at (104.0, 60.8)
- added P29: Conn_01x01_Pin, Connector_PinHeader_1.00mm:PinHeader_1x01_P1.00mm_Vertical, F.Cu at (106.3, 60.8)
- added P3: Conn_01x01_Pin, Connector_PinHeader_1.00mm:PinHeader_1x01_P1.00mm_Vertical, F.Cu at (74.1, 58.1)
- added P30: Conn_01x01_Pin, Connector_PinHeader_1.00mm:PinHeader_1x01_P1.00mm_Vertical, F.Cu at (108.6, 60.8)
- added P31: Conn_01x01_Pin, Connector_PinHeader_1.00mm:PinHeader_1x01_P1.00mm_Vertical, F.Cu at (110.9, 60.8)
- added P32: Conn_01x01_Pin, Connector_PinHeader_1.00mm:PinHeader_1x01_P1.00mm_Vertical, F.Cu at (110.9, 58.4)
- added P33: Conn_01x01_Pin, Connector_PinHeader_1.00mm:PinHeader_1x01_P1.00mm_Vertical, F.Cu at (113.5, 60.8)
- added P34: Conn_01x01_Pin, Connector_PinHeader_1.00mm:PinHeader_1x01_P1.00mm_Vertical, F.Cu at (113.5, 58.4)
- added P35: Conn_01x01_Pin, Connector_PinHeader_1.00mm:PinHeader_1x01_P1.00mm_Vertical, F.Cu at (115.8, 60.8)
- added P36: Conn_01x01_Pin, Connector_PinHeader_1.00mm:PinHeader_1x01_P1.00mm_Vertical, F.Cu at (115.8, 58.4)
- added P37: Conn_01x01_Pin, Connector_PinHeader_1.00mm:PinHeader_1x01_P1.00mm_Vertical, F.Cu at (118.1, 60.8)
- added P38: Conn_01x01_Pin, Connector_PinHeader_1.00mm:PinHeader_1x01_P1.00mm_Vertical, F.Cu at (118.1, 58.4)
- added P39: Conn_01x01_Pin, Connector_PinHeader_1.00mm:PinHeader_1x01_P1.00mm_Vertical, F.Cu at (120.4, 60.8)
- added P4: Conn_01x01_Pin, Connector_PinHeader_1.00mm:PinHeader_1x01_P1.00mm_Vertical, F.Cu at (74.1, 55.4)
- added P40: Conn_01x01_Pin, Connector_PinHeader_1.00mm:PinHeader_1x01_P1.00mm_Vertical, F.Cu at (120.4, 58.4)
- added P41: Conn_01x01_Pin, Connector_PinHeader_1.00mm:PinHeader_1x01_P1.00mm_Vertical, F.Cu at (122.7, 60.8)
- added P42: Conn_01x01_Pin, Connector_PinHeader_1.00mm:PinHeader_1x01_P1.00mm_Vertical, F.Cu at (122.7, 58.4)
- added P43: Conn_01x01_Pin, Connector_PinHeader_1.00mm:PinHeader_1x01_P1.00mm_Vertical, F.Cu at (125.0, 58.0)
- added P44: Conn_01x01_Pin, Connector_PinHeader_1.00mm:PinHeader_1x01_P1.00mm_Vertical, F.Cu at (125.0, 55.4)
- added P45: Conn_01x01_Pin, Connector_PinHeader_1.00mm:PinHeader_1x01_P1.00mm_Vertical, F.Cu at (127.3, 58.0)
- added P46: Conn_01x01_Pin, Connector_PinHeader_1.00mm:PinHeader_1x01_P1.00mm_Vertical, F.Cu at (127.3, 55.4)
- added P47: Conn_01x01_Pin, Connector_PinHeader_1.00mm:PinHeader_1x01_P1.00mm_Vertical, F.Cu at (129.6, 58.0)
- added P48: Conn_01x01_Pin, Connector_PinHeader_1.00mm:PinHeader_1x01_P1.00mm_Vertical, F.Cu at (129.6, 55.4)
- added P49: Conn_01x01_Pin, Connector_PinHeader_1.00mm:PinHeader_1x01_P1.00mm_Vertical, F.Cu at (131.9, 58.0)
- added P5: Conn_01x01_Pin, Connector_PinHeader_1.00mm:PinHeader_1x01_P1.00mm_Vertical, F.Cu at (76.4, 58.1)
- added P50: Conn_01x01_Pin, Connector_PinHeader_1.00mm:PinHeader_1x01_P1.00mm_Vertical, F.Cu at (131.9, 55.4)
- added P51: Conn_01x01_Pin, Connector_PinHeader_1.00mm:PinHeader_1x01_P1.00mm_Vertical, F.Cu at (133.3, 49.6)
- added P52: Conn_01x01_Pin, Connector_PinHeader_1.00mm:PinHeader_1x01_P1.00mm_Vertical, F.Cu at (131.0, 49.6)
- added P53: Conn_01x01_Pin, Connector_PinHeader_1.00mm:PinHeader_1x01_P1.00mm_Vertical, F.Cu at (128.7, 49.6)
- added P54: Conn_01x01_Pin, Connector_PinHeader_1.00mm:PinHeader_1x01_P1.00mm_Vertical, F.Cu at (126.4, 49.6)
- added P55: Conn_01x01_Pin, Connector_PinHeader_1.00mm:PinHeader_1x01_P1.00mm_Vertical, F.Cu at (124.1, 49.6)
- added P56: Conn_01x01_Pin, Connector_PinHeader_1.00mm:PinHeader_1x01_P1.00mm_Vertical, F.Cu at (121.8, 49.6)
- added P57: Conn_01x01_Pin, Connector_PinHeader_1.00mm:PinHeader_1x01_P1.00mm_Vertical, F.Cu at (119.5, 49.6)
- added P58: Conn_01x01_Pin, Connector_PinHeader_1.00mm:PinHeader_1x01_P1.00mm_Vertical, F.Cu at (117.2, 49.6)
- added P59: Conn_01x01_Pin, Connector_PinHeader_1.00mm:PinHeader_1x01_P1.00mm_Vertical, F.Cu at (117.2, 47.2)
- added P6: Conn_01x01_Pin, Connector_PinHeader_1.00mm:PinHeader_1x01_P1.00mm_Vertical, F.Cu at (76.4, 55.4)
- added P60: Conn_01x01_Pin, Connector_PinHeader_1.00mm:PinHeader_1x01_P1.00mm_Vertical, F.Cu at (119.5, 47.2)
- added P61: Conn_01x01_Pin, Connector_PinHeader_1.00mm:PinHeader_1x01_P1.00mm_Vertical, F.Cu at (121.8, 47.2)
- added P62: Conn_01x01_Pin, Connector_PinHeader_1.00mm:PinHeader_1x01_P1.00mm_Vertical, F.Cu at (124.1, 47.2)
- added P63: Conn_01x01_Pin, Connector_PinHeader_1.00mm:PinHeader_1x01_P1.00mm_Vertical, F.Cu at (126.4, 47.2)
- added P64: Conn_01x01_Pin, Connector_PinHeader_1.00mm:PinHeader_1x01_P1.00mm_Vertical, F.Cu at (128.7, 47.2)
- added P65: Conn_01x01_Pin, Connector_PinHeader_1.00mm:PinHeader_1x01_P1.00mm_Vertical, F.Cu at (131.0, 47.2)
- added P66: Conn_01x01_Pin, Connector_PinHeader_1.00mm:PinHeader_1x01_P1.00mm_Vertical, F.Cu at (133.3, 47.2)
- added P67: Conn_01x01_Pin, Connector_PinHeader_1.00mm:PinHeader_1x01_P1.00mm_Vertical, F.Cu at (117.3, 43.9)
- added P68: Conn_01x01_Pin, Connector_PinHeader_1.00mm:PinHeader_1x01_P1.00mm_Vertical, F.Cu at (119.6, 43.9)
- added P69: Conn_01x01_Pin, Connector_PinHeader_1.00mm:PinHeader_1x01_P1.00mm_Vertical, F.Cu at (121.9, 43.9)
- added P7: Conn_01x01_Pin, Connector_PinHeader_1.00mm:PinHeader_1x01_P1.00mm_Vertical, F.Cu at (78.7, 58.1)
- added P70: Conn_01x01_Pin, Connector_PinHeader_1.00mm:PinHeader_1x01_P1.00mm_Vertical, F.Cu at (124.2, 43.9)
- added P71: Conn_01x01_Pin, Connector_PinHeader_1.00mm:PinHeader_1x01_P1.00mm_Vertical, F.Cu at (126.5, 43.9)
- added P72: Conn_01x01_Pin, Connector_PinHeader_1.00mm:PinHeader_1x01_P1.00mm_Vertical, F.Cu at (128.8, 43.9)
- added P73: Conn_01x01_Pin, Connector_PinHeader_1.00mm:PinHeader_1x01_P1.00mm_Vertical, F.Cu at (131.1, 43.9)
- added P74: Conn_01x01_Pin, Connector_PinHeader_1.00mm:PinHeader_1x01_P1.00mm_Vertical, F.Cu at (117.4, 40.6)
- added P75: Conn_01x01_Pin, Connector_PinHeader_1.00mm:PinHeader_1x01_P1.00mm_Vertical, F.Cu at (119.7, 40.6)
- added P76: Conn_01x01_Pin, Connector_PinHeader_1.00mm:PinHeader_1x01_P1.00mm_Vertical, F.Cu at (74.3, 37.8)
- added P77: Conn_01x01_Pin, Connector_PinHeader_1.00mm:PinHeader_1x01_P1.00mm_Vertical, F.Cu at (74.2, 40.1)
- added P78: Conn_01x01_Pin, Connector_PinHeader_1.00mm:PinHeader_1x01_P1.00mm_Vertical, F.Cu at (76.5, 40.1)
- added P79: Conn_01x01_Pin, Connector_PinHeader_1.00mm:PinHeader_1x01_P1.00mm_Vertical, F.Cu at (78.8, 40.1)
- added P8: Conn_01x01_Pin, Connector_PinHeader_1.00mm:PinHeader_1x01_P1.00mm_Vertical, F.Cu at (78.7, 55.4)
- added P80: Conn_01x01_Pin, Connector_PinHeader_1.00mm:PinHeader_1x01_P1.00mm_Vertical, F.Cu at (81.1, 40.1)
- added P81: Conn_01x01_Pin, Connector_PinHeader_1.00mm:PinHeader_1x01_P1.00mm_Vertical, F.Cu at (83.4, 40.1)
- added P82: Conn_01x01_Pin, Connector_PinHeader_1.00mm:PinHeader_1x01_P1.00mm_Vertical, F.Cu at (85.7, 40.1)
- added P83: Conn_01x01_Pin, Connector_PinHeader_1.00mm:PinHeader_1x01_P1.00mm_Vertical, F.Cu at (88.0, 40.1)
- added P84: Conn_01x01_Pin, Connector_PinHeader_1.00mm:PinHeader_1x01_P1.00mm_Vertical, F.Cu at (74.2, 42.4)
- added P85: Conn_01x01_Pin, Connector_PinHeader_1.00mm:PinHeader_1x01_P1.00mm_Vertical, F.Cu at (76.5, 42.4)
- added P86: Conn_01x01_Pin, Connector_PinHeader_1.00mm:PinHeader_1x01_P1.00mm_Vertical, F.Cu at (78.8, 42.4)
- added P87: Conn_01x01_Pin, Connector_PinHeader_1.00mm:PinHeader_1x01_P1.00mm_Vertical, F.Cu at (81.1, 42.4)
- added P88: Conn_01x01_Pin, Connector_PinHeader_1.00mm:PinHeader_1x01_P1.00mm_Vertical, F.Cu at (83.4, 43.5)
- added P89: Conn_01x01_Pin, Connector_PinHeader_1.00mm:PinHeader_1x01_P1.00mm_Vertical, F.Cu at (85.7, 43.5)
- added P9: Conn_01x01_Pin, Connector_PinHeader_1.00mm:PinHeader_1x01_P1.00mm_Vertical, F.Cu at (81.0, 58.1)
- added P90: Conn_01x01_Pin, Connector_PinHeader_1.00mm:PinHeader_1x01_P1.00mm_Vertical, F.Cu at (88.0, 43.5)
- added P91: Conn_01x01_Pin, Connector_PinHeader_1.00mm:PinHeader_1x01_P1.00mm_Vertical, F.Cu at (88.0, 45.7)
- added P92: Conn_01x01_Pin, Connector_PinHeader_1.00mm:PinHeader_1x01_P1.00mm_Vertical, F.Cu at (85.7, 45.9)
- added P93: Conn_01x01_Pin, Connector_PinHeader_1.00mm:PinHeader_1x01_P1.00mm_Vertical, F.Cu at (83.4, 45.9)
- added P94: Conn_01x01_Pin, Connector_PinHeader_1.00mm:PinHeader_1x01_P1.00mm_Vertical, F.Cu at (81.1, 44.9)
- added P95: Conn_01x01_Pin, Connector_PinHeader_1.00mm:PinHeader_1x01_P1.00mm_Vertical, F.Cu at (78.8, 44.9)
- added P96: Conn_01x01_Pin, Connector_PinHeader_1.00mm:PinHeader_1x01_P1.00mm_Vertical, F.Cu at (78.8, 46.9)
- added P97: Conn_01x01_Pin, Connector_PinHeader_1.00mm:PinHeader_1x01_P1.00mm_Vertical, F.Cu at (76.5, 44.9)
- added P98: Conn_01x01_Pin, Connector_PinHeader_1.00mm:PinHeader_1x01_P1.00mm_Vertical, F.Cu at (76.5, 46.9)
- added P99: Conn_01x01_Pin, Connector_PinHeader_1.00mm:PinHeader_1x01_P1.00mm_Vertical, F.Cu at (74.2, 44.9)
- added R4: 330, Resistor_SMD:R_0603_1608Metric, F.Cu at (107.6, 37.7)
- added REF**: Fiducial_0.5mm_Mask1.5mm, Fiducial:Fiducial_0.5mm_Mask1.5mm, F.Cu at (134.4, 38.5)
- D2: value LED_G -> LED_GRE
- Daughter_Card_PIN1: footprint Connector_PCBEdge:SODIMM-200_1.8V_Card_edge -> MOSBius_V2_CHIP:SODIMM-200_1.8V_Card_edge_Extend
- moved D2 35.0 mm to (112.2, 37.7), turned to 180 degrees
- moved C6 22.3 mm to (73.8, 49.4), turned to -90 degrees
- moved MOSbius_V2 14.6 mm to (101.5, 48.4)
- moved Daughter_Card_PIN1 1.17 mm to (72.1, 66.6)
- renumbered MOSbius_V1 to MOSbius_V2
Connections:
- Daughter_Card_PIN1 pad 10: GND -> /DCC4_P_G_R_CC
- Daughter_Card_PIN1 pad 100: /DCC3_P_D_R_CC -> GND
- Daughter_Card_PIN1 pad 101: /DCC4_N_G_L_CS -> GND
- Daughter_Card_PIN1 pad 102: /DCC3_P_D_R_CS -> GND
- Daughter_Card_PIN1 pad 103: /DCC4_N_G_R_CC -> GND
- Daughter_Card_PIN1 pad 104: /DCC3_P_D_L_CC -> GND
- Daughter_Card_PIN1 pad 105: /DCC4_N_G_R_CS -> GND
- Daughter_Card_PIN1 pad 106: /DCC3_P_D_L_CS -> GND
- Daughter_Card_PIN1 pad 107: /DCC4_N_D_L_CC -> GND
- Daughter_Card_PIN1 pad 108: /DCC3_P_G_R_CC -> GND
- Daughter_Card_PIN1 pad 109: /DCC4_N_D_L_CS -> GND
- Daughter_Card_PIN1 pad 11: GND -> /SBUS4
- Daughter_Card_PIN1 pad 110: /DCC3_P_G_R_CS -> GND
- Daughter_Card_PIN1 pad 111: /DCC4_N_D_R_CC -> GND
- Daughter_Card_PIN1 pad 112: /DCC3_P_G_L_CC -> GND
- Daughter_Card_PIN1 pad 113: /DCC4_N_D_R_CS -> GND
- Daughter_Card_PIN1 pad 114: /DCC3_P_G_L_CS -> GND
- Daughter_Card_PIN1 pad 115: /DCC2_N_G_L_CC -> GND
- Daughter_Card_PIN1 pad 116: /CC_N_D_CS -> GND
- Daughter_Card_PIN1 pad 117: /DCC2_N_G_L_CS -> GND
- Daughter_Card_PIN1 pad 118: /ISINK_REF -> GND
- Daughter_Card_PIN1 pad 119: /DCC2_N_G_R_CC -> GND
- Daughter_Card_PIN1 pad 12: GND -> /DCC4_P_G_R_CS
- Daughter_Card_PIN1 pad 120: /CC_N_G_CS -> GND
- Daughter_Card_PIN1 pad 121: /DCC2_N_G_R_CS -> GND
- Daughter_Card_PIN1 pad 122: /CC_N_G_CC -> GND
- Daughter_Card_PIN1 pad 123: /DCC2_N_D_L_CC -> GND
- Daughter_Card_PIN1 pad 124: /CC_P_D_CC -> GND
- Daughter_Card_PIN1 pad 125: /DCC2_N_D_L_CS -> GND
- Daughter_Card_PIN1 pad 126: /CC_P_D_CS -> GND
- Daughter_Card_PIN1 pad 127: /DCC2_N_D_R_CC -> GND
- Daughter_Card_PIN1 pad 128: /CC_P_G_CC -> GND
- Daughter_Card_PIN1 pad 129: /DCC2_N_D_R_CS -> GND
- Daughter_Card_PIN1 pad 13: GND -> /SBUS3
- Daughter_Card_PIN1 pad 130: /CC_P_G_CS -> GND
- Daughter_Card_PIN1 pad 131: /DCC1_N_G_L_CC -> GND
- Daughter_Card_PIN1 pad 132: /DINV1_OUT_R -> GND
- Daughter_Card_PIN1 pad 133: /DCC1_N_G_L_CS -> GND
- Daughter_Card_PIN1 pad 134: /DINV1_INN_R -> GND
- Daughter_Card_PIN1 pad 135: /DCC1_N_G_R_CC -> GND
- Daughter_Card_PIN1 pad 136: /DINV1_INP_R -> GND
- Daughter_Card_PIN1 pad 137: /DCC1_N_G_R_CS -> GND
- Daughter_Card_PIN1 pad 138: /DINV1_OUT_L -> GND
- Daughter_Card_PIN1 pad 139: /DCC1_N_D_L_CC -> GND
- Daughter_Card_PIN1 pad 14: GND -> /DCC4_P_G_L_CC
- Daughter_Card_PIN1 pad 140: /DINV1_INN_L -> GND
- Daughter_Card_PIN1 pad 141: /DCC1_N_D_L_CS -> GND
- Daughter_Card_PIN1 pad 142: /DINV1_INP_L -> GND
- Daughter_Card_PIN1 pad 143: /DCC1_N_D_R_CC -> GND
- Daughter_Card_PIN1 pad 144: /DINV2_OUT_R -> GND
- Daughter_Card_PIN1 pad 145: /DCC1_N_D_R_CS -> GND
- Daughter_Card_PIN1 pad 146: /DINV2_INN_R -> GND
- Daughter_Card_PIN1 pad 147: /DINV2_INP_L -> GND
- Daughter_Card_PIN1 pad 148: /DINV2_INP_R -> GND
- Daughter_Card_PIN1 pad 149: /DINV2_INN_L -> GND
- Daughter_Card_PIN1 pad 15: GND -> /SBUS2
- Daughter_Card_PIN1 pad 150: /DINV2_OUT_L -> GND
- Daughter_Card_PIN1 pad 152: GND -> /DCC3_P_D_R_CS
- Daughter_Card_PIN1 pad 154: GND -> /DCC3_P_D_L_CC
- Daughter_Card_PIN1 pad 156: GND -> /DCC3_P_D_L_CS
- Daughter_Card_PIN1 pad 158: GND -> /DCC3_P_G_R_CC
- Daughter_Card_PIN1 pad 16: GND -> /DCC4_P_G_L_CS
- Daughter_Card_PIN1 pad 160: GND -> /DCC3_P_G_R_CS
- Daughter_Card_PIN1 pad 161: GND -> /DCC4_N_D_R_CC
- Daughter_Card_PIN1 pad 162: GND -> /DCC3_P_G_L_CC
- Daughter_Card_PIN1 pad 163: GND -> /DCC4_N_D_R_CS
- Daughter_Card_PIN1 pad 164: GND -> /DCC3_P_G_L_CS
- Daughter_Card_PIN1 pad 165: GND -> /DCC2_N_G_L_CC
- Daughter_Card_PIN1 pad 166: GND -> /CC_N_D_CS
- Daughter_Card_PIN1 pad 167: GND -> /DCC2_N_G_L_CS
- Daughter_Card_PIN1 pad 168: GND -> /CC_N_D_CC
- Daughter_Card_PIN1 pad 169: GND -> /DCC2_N_G_R_CC
- Daughter_Card_PIN1 pad 17: GND -> /SBUS1
- Daughter_Card_PIN1 pad 170: GND -> /CC_N_G_CS
- Daughter_Card_PIN1 pad 171: GND -> /DCC2_N_G_R_CS
- Daughter_Card_PIN1 pad 172: GND -> /CC_N_G_CC
- Daughter_Card_PIN1 pad 173: GND -> /DCC2_N_D_L_CC
- Daughter_Card_PIN1 pad 174: GND -> /CC_P_D_CC
- Daughter_Card_PIN1 pad 175: GND -> /DCC2_N_D_L_CS
- Daughter_Card_PIN1 pad 176: GND -> /CC_P_D_CS
- Daughter_Card_PIN1 pad 177: GND -> /DCC2_N_D_R_CC
- Daughter_Card_PIN1 pad 178: GND -> /CC_P_G_CC
- Daughter_Card_PIN1 pad 179: GND -> /DCC2_N_D_R_CS
- Daughter_Card_PIN1 pad 18: GND -> /DCC1_P_D_R_CC
- Daughter_Card_PIN1 pad 180: GND -> /CC_P_G_CS
- Daughter_Card_PIN1 pad 181: GND -> /DCC1_N_G_L_CC
- Daughter_Card_PIN1 pad 182: GND -> /DINV1_OUT_R
- Daughter_Card_PIN1 pad 183: GND -> /DCC1_N_G_L_CS
- Daughter_Card_PIN1 pad 184: GND -> /DINV1_INN_R
- Daughter_Card_PIN1 pad 185: GND -> /DCC1_N_G_R_CC
- Daughter_Card_PIN1 pad 186: GND -> /DINV1_INP_R
- Daughter_Card_PIN1 pad 187: GND -> /DCC1_N_G_R_CS
- Daughter_Card_PIN1 pad 188: GND -> /DINV1_OUT_L
- Daughter_Card_PIN1 pad 189: GND -> /DCC1_N_D_L_CC
- Daughter_Card_PIN1 pad 19: GND -> /OTA_P_INN
- Daughter_Card_PIN1 pad 190: GND -> /DINV1_INN_L
- Daughter_Card_PIN1 pad 191: GND -> /DCC1_N_D_L_CS
- Daughter_Card_PIN1 pad 192: GND -> /DINV1_INP_L
- Daughter_Card_PIN1 pad 193: GND -> /DCC1_N_D_R_CC
- Daughter_Card_PIN1 pad 194: GND -> /DINV2_OUT_R
- Daughter_Card_PIN1 pad 195: GND -> /DCC1_N_D_R_CS
- Daughter_Card_PIN1 pad 196: GND -> /DINV2_INN_R
- Daughter_Card_PIN1 pad 197: GND -> /DINV2_INP_L
- Daughter_Card_PIN1 pad 198: GND -> /DINV2_INP_R
- Daughter_Card_PIN1 pad 199: GND -> /DINV2_INN_L
- Daughter_Card_PIN1 pad 2: GND -> /DCC4_P_D_R_CC
- Daughter_Card_PIN1 pad 20: GND -> /DCC1_P_D_R_CS
- Daughter_Card_PIN1 pad 200: GND -> /DINV2_OUT_L
- Daughter_Card_PIN1 pad 21: GND -> /OTA_P_INP
- Daughter_Card_PIN1 pad 22: GND -> /DCC1_P_D_L_CC
- Daughter_Card_PIN1 pad 23: GND -> /OTA_P_OUT
- Daughter_Card_PIN1 pad 24: GND -> /DCC1_P_D_L_CS
- Daughter_Card_PIN1 pad 25: GND -> VDD
- Daughter_Card_PIN1 pad 26: GND -> /DCC1_P_G_R_CC
- Daughter_Card_PIN1 pad 27: GND -> /OTA_N_INP
- Daughter_Card_PIN1 pad 28: GND -> /DCC1_P_G_R_CS
- Daughter_Card_PIN1 pad 29: GND -> /OTA_N_INN
- Daughter_Card_PIN1 pad 3: GND -> /EN
- Daughter_Card_PIN1 pad 30: GND -> /DCC1_P_G_L_CC
- Daughter_Card_PIN1 pad 31: GND -> /OTA_N_OUT
- Daughter_Card_PIN1 pad 32: GND -> /DCC1_P_G_L_CS
- Daughter_Card_PIN1 pad 33: GND -> /DCC3_N_G_L_CC
- Daughter_Card_PIN1 pad 34: GND -> /DCC2_P_D_R_CC
- Daughter_Card_PIN1 pad 35: GND -> /DCC3_N_G_L_CS
- Daughter_Card_PIN1 pad 36: GND -> /DCC2_P_D_R_CS
- Daughter_Card_PIN1 pad 37: GND -> /DCC3_N_G_R_CC
- Daughter_Card_PIN1 pad 38: GND -> /DCC2_P_D_L_CC
- Daughter_Card_PIN1 pad 39: GND -> /DCC3_N_G_R_CS
- Daughter_Card_PIN1 pad 4: GND -> /DCC4_P_D_R_CS
- Daughter_Card_PIN1 pad 40: GND -> /DCC2_P_D_L_CS
- Daughter_Card_PIN1 pad 41: GND -> /DCC3_N_D_L_CC
- Daughter_Card_PIN1 pad 42: GND -> /DCC2_P_G_R_CC
- Daughter_Card_PIN1 pad 43: GND -> /DCC3_N_D_L_CS
- Daughter_Card_PIN1 pad 44: GND -> /DCC2_P_G_R_CS
- Daughter_Card_PIN1 pad 45: GND -> /DCC3_N_D_R_CC
- Daughter_Card_PIN1 pad 46: GND -> /DCC2_P_G_L_CC
- Daughter_Card_PIN1 pad 47: GND -> /DCC3_N_D_R_CS
- Daughter_Card_PIN1 pad 48: GND -> /DCC2_P_G_L_CS
- Daughter_Card_PIN1 pad 49: GND -> /DCC4_N_G_L_CC
- Daughter_Card_PIN1 pad 5: GND -> /CLK
- Daughter_Card_PIN1 pad 50: GND -> /DCC3_P_D_R_CC
- Daughter_Card_PIN1 pad 51: GND -> /DCC4_N_G_L_CS
- Daughter_Card_PIN1 pad 52: /DCC4_P_D_R_CC -> GND
- Daughter_Card_PIN1 pad 53: /EN -> /DCC4_N_G_R_CC
- Daughter_Card_PIN1 pad 54: /DCC4_P_D_R_CS -> GND
- Daughter_Card_PIN1 pad 55: /CLK -> /DCC4_N_G_R_CS
- Daughter_Card_PIN1 pad 56: /DCC4_P_D_L_CC -> GND
- Daughter_Card_PIN1 pad 57: /DATA_SBUS6 -> /DCC4_N_D_L_CC
- Daughter_Card_PIN1 pad 58: /DCC4_P_D_L_CS -> GND
- Daughter_Card_PIN1 pad 59: /SBUS5 -> /DCC4_N_D_L_CS
- Daughter_Card_PIN1 pad 6: GND -> /DCC4_P_D_L_CC
- Daughter_Card_PIN1 pad 60: /DCC4_P_G_R_CC -> GND
- Daughter_Card_PIN1 pad 61: /SBUS4 -> GND
- Daughter_Card_PIN1 pad 62: /DCC4_P_G_R_CS -> GND
- Daughter_Card_PIN1 pad 63: /SBUS3 -> GND
- Daughter_Card_PIN1 pad 64: /DCC4_P_G_L_CC -> GND
- Daughter_Card_PIN1 pad 65: /SBUS2 -> GND
- Daughter_Card_PIN1 pad 66: /DCC4_P_G_L_CS -> GND
- Daughter_Card_PIN1 pad 67: /SBUS1 -> GND
- Daughter_Card_PIN1 pad 68: /DCC1_P_D_R_CC -> GND
- Daughter_Card_PIN1 pad 69: /OTA_P_INN -> GND
- Daughter_Card_PIN1 pad 7: GND -> /DATA_SBUS6
- Daughter_Card_PIN1 pad 70: /DCC1_P_D_R_CS -> GND
- Daughter_Card_PIN1 pad 71: /OTA_P_INP -> GND
- Daughter_Card_PIN1 pad 72: /DCC1_P_D_L_CC -> GND
- Daughter_Card_PIN1 pad 73: /OTA_P_OUT -> GND
- Daughter_Card_PIN1 pad 74: /DCC1_P_D_L_CS -> GND
- Daughter_Card_PIN1 pad 75: VDD -> GND
- Daughter_Card_PIN1 pad 76: /DCC1_P_G_R_CC -> GND
- Daughter_Card_PIN1 pad 77: /OTA_N_INP -> GND
- Daughter_Card_PIN1 pad 78: /DCC1_P_G_R_CS -> GND
- Daughter_Card_PIN1 pad 79: /OTA_N_INN -> GND
- Daughter_Card_PIN1 pad 8: GND -> /DCC4_P_D_L_CS
- Daughter_Card_PIN1 pad 80: /DCC1_P_G_L_CC -> GND
- Daughter_Card_PIN1 pad 81: /OTA_N_OUT -> GND
- Daughter_Card_PIN1 pad 82: /DCC1_P_G_L_CS -> GND
- Daughter_Card_PIN1 pad 83: /DCC3_N_G_L_CC -> GND
- Daughter_Card_PIN1 pad 84: /DCC2_P_D_R_CC -> GND
- Daughter_Card_PIN1 pad 85: /DCC3_N_G_L_CS -> GND
- Daughter_Card_PIN1 pad 86: /DCC2_P_D_R_CS -> GND
- Daughter_Card_PIN1 pad 87: /DCC3_N_G_R_CC -> GND
- Daughter_Card_PIN1 pad 88: /DCC2_P_D_L_CC -> GND
- Daughter_Card_PIN1 pad 89: /DCC3_N_G_R_CS -> GND
- Daughter_Card_PIN1 pad 9: GND -> /SBUS5
- Daughter_Card_PIN1 pad 90: /DCC2_P_D_L_CS -> GND
- Daughter_Card_PIN1 pad 91: /DCC3_N_D_L_CC -> GND
- Daughter_Card_PIN1 pad 92: /DCC2_P_G_R_CC -> GND
- Daughter_Card_PIN1 pad 93: /DCC3_N_D_L_CS -> GND
- Daughter_Card_PIN1 pad 94: /DCC2_P_G_R_CS -> GND
- Daughter_Card_PIN1 pad 95: /DCC3_N_D_R_CC -> GND
- Daughter_Card_PIN1 pad 96: /DCC2_P_G_L_CC -> GND
- Daughter_Card_PIN1 pad 97: /DCC3_N_D_R_CS -> GND
- Daughter_Card_PIN1 pad 98: /DCC2_P_G_L_CS -> GND
- Daughter_Card_PIN1 pad 99: /DCC4_N_G_L_CC -> GND
Routing:
- net GND: track 6.85 -> 112.8 mm, vias 0 -> 82
- net /CC_N_G_CS: track 0.00 -> 78.4 mm
- net /DCC3_P_D_L_CS: track 0.00 -> 77.7 mm
- net /DCC2_P_G_L_CS: track 0.00 -> 76.4 mm
- net /DCC3_P_D_R_CC: track 0.00 -> 74.9 mm
- net /CC_N_G_CC: track 0.00 -> 73.8 mm
- net /DCC2_P_D_R_CC: track 0.00 -> 73.4 mm
- net /DCC3_P_G_R_CC: track 0.00 -> 72.2 mm
- net /DCC2_P_G_L_CC: track 0.00 -> 70.6 mm
- net /CC_P_D_CC: track 0.00 -> 68.3 mm
- net /DCC1_P_G_L_CS: track 0.00 -> 68.2 mm
- net /DCC3_P_G_R_CS: track 0.00 -> 67.0 mm
- net /DCC2_P_G_R_CS: track 0.00 -> 65.1 mm
- net /DCC2_P_G_R_CC: track 0.00 -> 63.6 mm
- net /CC_P_D_CS: track 0.00 -> 63.5 mm
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- added copper zone on B.Cu, net GND
- added copper zone on F.Cu, net GND
Other:
- board size 67.6 x 25.4 mm -> 67.6 x 31.1 mm
- board text added: "20250912"
- board text added: "32.1mm"
- board text added: "MOSBius V2"
- board text added: "S/N"
- board text added: "https://mosbius.org"

Commit message: 0919
Connections:
- MOSbius_V2 pad : (no net) -> GND
Changed lines of the file:
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@@
 			(roundrect_rratio 0.125628)
 		)
+		(pad "" smd rect
+			(at 0.53855 -0.223075 45)
+			(size 7.4 7.4)
+			(property pad_prop_heatsink)
+			(layers "F.Cu" "F.Mask")
+			(net 1 "GND")
+			(zone_connect 2)
+		)
 		(pad "" smd roundrect
 			(at 0.53855 3.270033 45)
@@
 			(pintype "bidirectional")
 		)
-		(pad "101" smd rect
-			(at 0.53855 -0.223075 45)
-			(size 7.4 7.4)
-			(property pad_prop_heatsink)
-			(layers "F.Cu" "F.Mask")
-			(zone_connect 2)
-		)
 		(embedded_fonts no)
 		(model "${KICAD9_3DMODEL_DIR}/Package_DFN_QFN.3dshapes/ArtInChip_QFN-100-1EP_12x12mm_P0.4mm_EP7.4x7.4mm.step"
@@
 	(via
 		(at 95.4 48.3)
-		(size 0.6)
-		(drill 0.3)
+		(size 0.6096)
+		(drill 0.3048)
 		(layers "F.Cu" "B.Cu")
 		(net 2)
@@
 	(via
 		(at 104.8 39)
-		(size 0.6)
-		(drill 0.3)
+		(size 0.6096)
+		(drill 0.3048)
 		(layers "F.Cu" "B.Cu")
 		(net 2)
