File: Mother_Card/Mother_Card.kicad_pcb (KiCad board)
At the start: 2 copper layers, 45 parts, among them IC1 SN74LVC2G34DBVR, J1 5-1746530-4, J11 Conn_01x25_Pin, J12 Conn_01x02_Pin, J13 PINHD_1x2_Male, J14 PINHD_1x2_Male, J14_GND3 Conn_01x03, J18_VDC1 Conn_01x02, J2 PINHD_1x2_Male, J3 Conn_01x25_Pin, J4 Conn_01x25_Pin, J5 PINHD_1x2_Male, J6 Conn_02x03_Row_Letter_First, J7 PINHD_1x2_Male, J8 Conn_01x25_Pin, J9 PINHD_1x2_Male, U1 NCV8164ASN250T1G_LDO_2.5V

Commit message: update in 0912
Parts:
- removed C19, C22, C25: 1u, Capacitor_SMD:C_0603_1608Metric
- removed C20, C21, C24: 10u, Capacitor_SMD:C_0603_1608Metric
- removed C23, C26: 0.1u, Capacitor_SMD:C_0603_1608Metric
- removed J14_GND3: Conn_01x03, Connector_PinHeader_2.54mm:PinHeader_1x03_P2.54mm_Vertical
- removed J18_VDC1: Conn_01x02, Connector_PinHeader_2.54mm:PinHeader_1x02_P2.54mm_Vertical
- removed J4: Conn_01x25_Pin, Connector_PinHeader_2.54mm:PinHeader_1x25_P2.54mm_Vertical
- removed the J5 at (134.2, 113.5)
- removed JP1_LDOPG1: Jumper_2_Open, Connector_PinHeader_2.54mm:PinHeader_1x02_P2.54mm_Vertical
- removed R10: 10K, Resistor_SMD:R_0603_1608Metric
- removed R18: 1k, Resistor_SMD:R_0603_1608Metric
- removed R19: 330, Resistor_SMD:R_0603_1608Metric
- added ?: , , F.Cu at (215.3, 122.5)
- added C10: 1u, Capacitor_SMD:C_0603_1608Metric, F.Cu at (111.3, 93.1)
- added C12: 10u, Capacitor_SMD:C_0603_1608Metric, F.Cu at (111.3, 90.3)
- added C14: 1u, Capacitor_SMD:C_0603_1608Metric, F.Cu at (208.0, 124.7)
- added C15: 0.1u, Capacitor_SMD:C_0603_1608Metric, F.Cu at (209.9, 126.4)
- added C16: 0.1u, Capacitor_SMD:C_0603_1608Metric, F.Cu at (210.3, 64.1)
- added C9: 0.1u, Capacitor_SMD:C_0603_1608Metric, F.Cu at (91.2, 72.2)
- added D2: LED_GRE, MOSBius_V2_CHIP:LED_150120RS75000_WRE, F.Cu at (195.2, 89.0)
- added D3: LED_OR, MOSBius_V2_CHIP:LED_150120RS75000_WRE, F.Cu at (195.2, 80.7)
- added EN_TO_CHIP'1: PINHD_1x2_Male, Connector_PinHeader_2.54mm:PinHeader_1x02_P2.54mm_Vertical, F.Cu at (200.5, 97.3)
- added G***: LOGO, Custom_Footprints:logo4, F.Cu at (144.0, 78.0)
- added G***: LOGO, Custom_Footprints:logo4, F.Cu at (149.2, 108.2)
- added IC2: AD8542ARMZ-REEL, MOSBius_V2_CHIP:AD8542, F.Cu at (203.7, 81.5)
- added IC3: SN74LVC1G3157DBVR, MOSBius_V2_CHIP:SN74LVC1G3157, F.Cu at (184.7, 85.0)
- added J1: PINHD_1x2_Male, Connector_PinHeader_2.54mm:PinHeader_1x02_P2.54mm_Vertical, F.Cu at (110.5, 102.3)
- added J10: USB4736, Connector_USB:USB_C_Receptacle_GCT_USB4125-xx-x_6P_TopMnt_Horizontal, F.Cu at (90.0, 88.1)
- added J14_GND1: Conn_01x03, Connector_PinHeader_2.54mm:PinHeader_1x03_P2.54mm_Vertical, F.Cu at (101.2, 76.0)
- added J14_GND2: Conn_01x03, Connector_PinHeader_2.54mm:PinHeader_1x03_P2.54mm_Vertical, F.Cu at (96.3, 76.0)
- added J_CLK_RPI1: CLK_RPI, Connector_PinHeader_2.54mm:PinHeader_1x01_P2.54mm_Vertical, F.Cu at (195.5, 93.5)
- added J_DATA_RPI1: DATA_RPI, Connector_PinHeader_2.54mm:PinHeader_1x01_P2.54mm_Vertical, F.Cu at (189.9, 84.5)
- added J_VCM1: VCM, Connector_PinHeader_2.54mm:PinHeader_1x01_P2.54mm_Vertical, F.Cu at (201.5, 77.2)
- added OPAMP_1: Conn_01x03, Connector_PinHeader_2.54mm:PinHeader_1x03_P2.54mm_Vertical, F.Cu at (209.5, 76.2)
- added R2: 1k, Resistor_SMD:R_0603_1608Metric, F.Cu at (102.5, 101.6)
- added R3: 1k, Resistor_SMD:R_0603_1608Metric, F.Cu at (206.0, 87.3)
- added R4: 330, Resistor_SMD:R_0603_1608Metric, F.Cu at (190.2, 89.0)
- added R5: 330, Resistor_SMD:R_0603_1608Metric, F.Cu at (190.7, 80.7)
- added REF**: Fiducial_0.5mm_Mask1mm, Fiducial:Fiducial_0.5mm_Mask1mm, F.Cu at (88.5, 132.1)
- added REF**: Fiducial_0.5mm_Mask1mm, Fiducial:Fiducial_0.5mm_Mask1mm, F.Cu at (88.7, 76.0)
- added Rd_1: 5.1K, Resistor_SMD:R_0603_1608Metric, F.Cu at (107.3, 86.8)
- added Rd_2: 5.1K, Resistor_SMD:R_0603_1608Metric, F.Cu at (106.5, 90.3)
- added VDD_GND_RPI1: PINHD_1x2_Male, Connector_PinHeader_2.54mm:PinHeader_1x02_P2.54mm_Vertical, F.Cu at (200.4, 106.3)
- C1: value 1u -> 0.1u
- C11: value 10u -> 0.1u
- C13, C6: value 1u -> 10u
- C17, C3, C7: value 0.1u -> 1u
- C18: value 0.1u -> 10u
- D1: value LED_OR -> LED_BLUE
- IC1: value SN74LVC2G34DBVR -> SN74LVC1G3157DBVR; footprint MOSBius_V2_CHIP:SN74LVC2G34DBVR -> MOSBius_V2_CHIP:SN74LVC1G3157
- J12: value Conn_01x02_Pin -> Conn_01x25_Pin; footprint Connector_PinHeader_2.54mm:PinHeader_1x02_P2.54mm_Vertical -> Connector_PinHeader_2.54mm:PinHeader_1x25_P2.54mm_Vertical
- J13: value PINHD_1x2_Male -> Conn_01x02_Pin
- J3: value Conn_01x25_Pin -> PINHD_1x2_Male; footprint Connector_PinHeader_2.54mm:PinHeader_1x25_P2.54mm_Vertical -> Connector_PinHeader_2.54mm:PinHeader_1x02_P2.54mm_Vertical; moved to F.Cu
- J6: value Conn_02x03_Row_Letter_First -> PINHD_1x2_Male; footprint Connector_PinHeader_2.54mm:PinHeader_2x03_P2.54mm_Vertical -> Connector_PinHeader_2.54mm:PinHeader_1x02_P2.54mm_Vertical; moved to B.Cu
- J7: moved to B.Cu
- J9: value PINHD_1x2_Male -> Conn_01x25_Pin; footprint Connector_PinHeader_2.54mm:PinHeader_1x02_P2.54mm_Vertical -> Connector_PinHeader_2.54mm:PinHeader_1x25_P2.54mm_Vertical
- R1: value 25k -> 330
- moved J9 173.5 mm to (88.9, 136.9), turned to -90 degrees
- moved C3 156.9 mm to (99.5, 101.6), turned to 90 degrees
- moved C7 153.2 mm to (95.5, 70.2), turned to -90 degrees
- moved C6 152.1 mm to (99.6, 122.2), turned to -90 degrees
- moved C8 149.0 mm to (97.1, 124.3), turned to -90 degrees
- moved RV1 146.6 mm to (96.8, 110.1)
- moved C18 89.3 mm to (206.7, 64.1), turned to -90 degrees
- moved J8 85.4 mm to (149.9, 58.4), turned to 90 degrees
- moved C17 81.7 mm to (208.6, 64.1)
- moved RV2 81.1 mm to (211.8, 84.8), turned to 90 degrees
- moved C13 78.4 mm to (206.1, 123.0)
- moved C4 76.7 mm to (206.0, 88.9), turned to 0 degrees
- moved C2 69.5 mm to (206.0, 90.6), turned to 0 degrees
- moved J13 67.6 mm to (91.4, 66.0)
- moved J12 65.8 mm to (154.9, 136.9), turned to -90 degrees
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- renumbered J1 to J5
Connections:
- C2 pad 1: Net-(C1-Pad1) -> Net-(C2-Pad1)
- C3 pad 1: Net-(C3-Pad1) -> Net-(C1-Pad1)
- C4 pad 1: LDO_VIN -> Net-(C2-Pad1)
- C5 pad 1: LDO_VIN -> VDD
- C8 pad 1: Net-(C3-Pad1) -> VDD
- IC1 pad 1: CLK_PRE -> /CLK_SC
- IC1 pad 3: DATA_SBUS6_PRE -> Net-(IC1-B1)
- IC1 pad 4: /DATA_SBUS6 -> /CLK
- IC1 pad 6: /CLK -> /EN
- J11 pad 1: unconnected-(J11-Pin_1-Pad1) -> GND
- J11 pad 2: unconnected-(J11-Pin_2-Pad2) -> GND
- J11 pad 3: /CLK -> /CLK_SC
- J11 pad 4: /DATA_SBUS6 -> /SBUS6
- J12 pad 1: VDD -> /DCC3_P_D_R_CC
- J12 pad 2: GND -> /DCC2_P_G_L_CS
- J2 pad 1: Net-(C3-Pad1) -> Net-(C2-Pad1)
- J2 pad 2: VCM -> Net-(IC2-+IN_A)
- J3 pad 1: /DINV2_OUT_L -> Net-(J3-Pad1)
- J3 pad 2: /DINV2_INP_R -> Net-(C1-Pad1)
- J5 pad 10: GND -> /DCC4_P_G_R_CC
- J5 pad 100: /DCC3_P_D_R_CC -> GND
- J5 pad 101: /DCC4_N_G_L_CS -> GND
- J5 pad 102: /DCC3_P_D_R_CS -> GND
- J5 pad 103: /DCC4_N_G_R_CC -> GND
- J5 pad 104: /DCC3_P_D_L_CC -> GND
- J5 pad 105: /DCC4_N_G_R_CS -> GND
- J5 pad 106: /DCC3_P_D_L_CS -> GND
- J5 pad 107: /DCC4_N_D_L_CC -> GND
- J5 pad 108: /DCC3_P_G_R_CC -> GND
- J5 pad 109: /DCC4_N_D_L_CS -> GND
- J5 pad 11: GND -> /SBUS4
- J5 pad 110: /DCC3_P_G_R_CS -> GND
- J5 pad 111: /DCC4_N_D_R_CC -> GND
- J5 pad 112: /DCC3_P_G_L_CC -> GND
- J5 pad 113: /DCC4_N_D_R_CS -> GND
- J5 pad 114: /DCC3_P_G_L_CS -> GND
- J5 pad 115: /DCC2_N_G_L_CC -> GND
- J5 pad 116: /CC_N_D_CS -> GND
- J5 pad 117: /DCC2_N_G_L_CS -> GND
- J5 pad 118: ISINK_REF -> GND
- J5 pad 119: /DCC2_N_G_R_CC -> GND
- J5 pad 12: GND -> /DCC4_P_G_R_CS
- J5 pad 120: /CC_N_G_CS -> GND
- J5 pad 121: /DCC2_N_G_R_CS -> GND
- J5 pad 122: /CC_N_G_CC -> GND
- J5 pad 123: /DCC2_N_D_L_CC -> GND
- J5 pad 124: /CC_P_D_CC -> GND
- J5 pad 125: /DCC2_N_D_L_CS -> GND
- J5 pad 126: /CC_P_D_CS -> GND
- J5 pad 127: /DCC2_N_D_R_CC -> GND
- J5 pad 128: /CC_P_G_CC -> GND
- J5 pad 129: /DCC2_N_D_R_CS -> GND
- J5 pad 13: GND -> /SBUS3
- J5 pad 130: /CC_P_G_CS -> GND
- J5 pad 131: /DCC1_N_G_L_CC -> GND
- J5 pad 132: /DINV1_OUT_R -> GND
- J5 pad 133: /DCC1_N_G_L_CS -> GND
- J5 pad 134: /DINV1_INN_R -> GND
- J5 pad 135: /DCC1_N_G_R_CC -> GND
- J5 pad 136: /DINV1_INP_R -> GND
- J5 pad 137: /DCC1_N_G_R_CS -> GND
- J5 pad 138: /DINV1_OUT_L -> GND
- J5 pad 139: /DCC1_N_D_L_CC -> GND
- J5 pad 14: GND -> /DCC4_P_G_L_CC
- J5 pad 140: /DINV1_INN_L -> GND
- J5 pad 141: /DCC1_N_D_L_CS -> GND
- J5 pad 142: /DINV1_INP_L -> GND
- J5 pad 143: /DCC1_N_D_R_CC -> GND
- J5 pad 144: /DINV2_OUT_R -> GND
- J5 pad 145: /DCC1_N_D_R_CS -> GND
- J5 pad 146: /DINV2_INN_R -> GND
- J5 pad 147: /DINV2_INP_L -> GND
- J5 pad 148: /DINV2_INP_R -> GND
- J5 pad 149: /DINV2_INN_L -> GND
- J5 pad 15: GND -> /SBUS2
- J5 pad 150: /DINV2_OUT_L -> GND
- J5 pad 152: GND -> /DCC3_P_D_R_CS
- J5 pad 154: GND -> /DCC3_P_D_L_CC
- J5 pad 156: GND -> /DCC3_P_D_L_CS
- J5 pad 158: GND -> /DCC3_P_G_R_CC
- J5 pad 16: GND -> /DCC4_P_G_L_CS
- J5 pad 160: GND -> /DCC3_P_G_R_CS
- J5 pad 161: GND -> /DCC4_N_D_R_CC
- J5 pad 162: GND -> /DCC3_P_G_L_CC
- J5 pad 163: GND -> /DCC4_N_D_R_CS
- J5 pad 164: GND -> /DCC3_P_G_L_CS
- J5 pad 165: GND -> /DCC2_N_G_L_CC
- J5 pad 166: GND -> /CC_N_D_CS
- J5 pad 167: GND -> /DCC2_N_G_L_CS
- J5 pad 168: GND -> ISINK_REF
- J5 pad 169: GND -> /DCC2_N_G_R_CC
- J5 pad 17: GND -> /SBUS1
- J5 pad 170: GND -> /CC_N_G_CS
- J5 pad 171: GND -> /DCC2_N_G_R_CS
- J5 pad 172: GND -> /CC_N_G_CC
- J5 pad 173: GND -> /DCC2_N_D_L_CC
- J5 pad 174: GND -> /CC_P_D_CC
- J5 pad 175: GND -> /DCC2_N_D_L_CS
- J5 pad 176: GND -> /CC_P_D_CS
- J5 pad 177: GND -> /DCC2_N_D_R_CC
- J5 pad 178: GND -> /CC_P_G_CC
- J5 pad 179: GND -> /DCC2_N_D_R_CS
- J5 pad 18: GND -> /DCC1_P_D_R_CC
- J5 pad 180: GND -> /CC_P_G_CS
- J5 pad 181: GND -> /DCC1_N_G_L_CC
- J5 pad 182: GND -> /DINV1_OUT_R
- J5 pad 183: GND -> /DCC1_N_G_L_CS
- J5 pad 184: GND -> /DINV1_INN_R
- J5 pad 185: GND -> /DCC1_N_G_R_CC
- J5 pad 186: GND -> /DINV1_INP_R
- J5 pad 187: GND -> /DCC1_N_G_R_CS
- J5 pad 188: GND -> /DINV1_OUT_L
- J5 pad 189: GND -> /DCC1_N_D_L_CC
- J5 pad 19: GND -> /OTA_P_INN
- J5 pad 190: GND -> /DINV1_INN_L
- J5 pad 191: GND -> /DCC1_N_D_L_CS
- J5 pad 192: GND -> /DINV1_INP_L
- J5 pad 193: GND -> /DCC1_N_D_R_CC
- J5 pad 194: GND -> /DINV2_OUT_R
- J5 pad 195: GND -> /DCC1_N_D_R_CS
- J5 pad 196: GND -> /DINV2_INN_R
- J5 pad 197: GND -> /DINV2_INP_L
- J5 pad 198: GND -> /DINV2_INP_R
- J5 pad 199: GND -> /DINV2_INN_L
- J5 pad 2: GND -> /DCC4_P_D_R_CC
- J5 pad 20: GND -> /DCC1_P_D_R_CS
- J5 pad 200: GND -> /DINV2_OUT_L
- J5 pad 21: GND -> /OTA_P_INP
- J5 pad 22: GND -> /DCC1_P_D_L_CC
- J5 pad 23: GND -> /OTA_P_OUT
- J5 pad 24: GND -> /DCC1_P_D_L_CS
- J5 pad 25: GND -> VDD
- J5 pad 26: GND -> /DCC1_P_G_R_CC
- J5 pad 27: GND -> /OTA_N_INP
- J5 pad 28: GND -> /DCC1_P_G_R_CS
- J5 pad 29: GND -> /OTA_N_INN
- J5 pad 3: GND -> /EN
- J5 pad 30: GND -> /DCC1_P_G_L_CC
- J5 pad 31: GND -> /OTA_N_OUT
- J5 pad 32: GND -> /DCC1_P_G_L_CS
- J5 pad 33: GND -> /DCC3_N_G_L_CC
- J5 pad 34: GND -> /DCC2_P_D_R_CC
- J5 pad 35: GND -> /DCC3_N_G_L_CS
- J5 pad 36: GND -> /DCC2_P_D_R_CS
- J5 pad 37: GND -> /DCC3_N_G_R_CC
- J5 pad 38: GND -> /DCC2_P_D_L_CC
- J5 pad 39: GND -> /DCC3_N_G_R_CS
- J5 pad 4: GND -> /DCC4_P_D_R_CS
- J5 pad 40: GND -> /DCC2_P_D_L_CS
- J5 pad 41: GND -> /DCC3_N_D_L_CC
- J5 pad 42: GND -> /DCC2_P_G_R_CC
- J5 pad 43: GND -> /DCC3_N_D_L_CS
- J5 pad 44: GND -> /DCC2_P_G_R_CS
- J5 pad 45: GND -> /DCC3_N_D_R_CC
- J5 pad 46: GND -> /DCC2_P_G_L_CC
- J5 pad 47: GND -> /DCC3_N_D_R_CS
- J5 pad 48: GND -> /DCC2_P_G_L_CS
- J5 pad 49: GND -> /DCC4_N_G_L_CC
- J5 pad 5: GND -> /CLK
- J5 pad 50: GND -> /DCC3_P_D_R_CC
- J5 pad 51: GND -> /DCC4_N_G_L_CS
- J5 pad 52: /DCC4_P_D_R_CC -> GND
- J5 pad 53: EN -> /DCC4_N_G_R_CC
- J5 pad 54: /DCC4_P_D_R_CS -> GND
- J5 pad 55: /CLK -> /DCC4_N_G_R_CS
- J5 pad 56: /DCC4_P_D_L_CC -> GND
- J5 pad 57: /DATA_SBUS6 -> /DCC4_N_D_L_CC
- J5 pad 58: /DCC4_P_D_L_CS -> GND
- J5 pad 59: /SBUS5 -> /DCC4_N_D_L_CS
- J5 pad 6: GND -> /DCC4_P_D_L_CC
- J5 pad 60: /DCC4_P_G_R_CC -> GND
- J5 pad 61: /SBUS4 -> GND
- J5 pad 62: /DCC4_P_G_R_CS -> GND
- J5 pad 63: /SBUS3 -> GND
- J5 pad 64: /DCC4_P_G_L_CC -> GND
- J5 pad 65: /SBUS2 -> GND
- J5 pad 66: /DCC4_P_G_L_CS -> GND
- J5 pad 67: /SBUS1 -> GND
- J5 pad 68: /DCC1_P_D_R_CC -> GND
- J5 pad 69: /OTA_P_INN -> GND
- J5 pad 7: GND -> /DATA_SBUS6
- J5 pad 70: /DCC1_P_D_R_CS -> GND
- J5 pad 71: /OTA_P_INP -> GND
- J5 pad 72: /DCC1_P_D_L_CC -> GND
- J5 pad 73: /OTA_P_OUT -> GND
- J5 pad 74: /DCC1_P_D_L_CS -> GND
- J5 pad 75: VDD -> GND
- J5 pad 76: /DCC1_P_G_R_CC -> GND
- J5 pad 77: /OTA_N_INP -> GND
- J5 pad 78: /DCC1_P_G_R_CS -> GND
- J5 pad 79: /OTA_N_INN -> GND
- J5 pad 8: GND -> /DCC4_P_D_L_CS
- J5 pad 80: /DCC1_P_G_L_CC -> GND
- J5 pad 81: /OTA_N_OUT -> GND
- J5 pad 82: /DCC1_P_G_L_CS -> GND
- J5 pad 83: /DCC3_N_G_L_CC -> GND
- J5 pad 84: /DCC2_P_D_R_CC -> GND
- J5 pad 85: /DCC3_N_G_L_CS -> GND
- J5 pad 86: /DCC2_P_D_R_CS -> GND
- J5 pad 87: /DCC3_N_G_R_CC -> GND
- J5 pad 88: /DCC2_P_D_L_CC -> GND
- J5 pad 89: /DCC3_N_G_R_CS -> GND
- J5 pad 9: GND -> /SBUS5
- J5 pad 90: /DCC2_P_D_L_CS -> GND
- J5 pad 91: /DCC3_N_D_L_CC -> GND
- J5 pad 92: /DCC2_P_G_R_CC -> GND
- J5 pad 93: /DCC3_N_D_L_CS -> GND
- J5 pad 94: /DCC2_P_G_R_CS -> GND
- J5 pad 95: /DCC3_N_D_R_CC -> GND
- J5 pad 96: /DCC2_P_G_L_CC -> GND
- J5 pad 97: /DCC3_N_D_R_CS -> GND
- J5 pad 98: /DCC2_P_G_L_CS -> GND
- J5 pad 99: /DCC4_N_G_L_CC -> GND
- J5 pad MP1: GND -> unconnected-(J5-PadMP1)
- J5 pad MP2: GND -> unconnected-(J5-PadMP2)
- J6 pad 1: (no net) -> VDD
- J6 pad 2: (no net) -> GND
- J7 pad 1: Net-(C1-Pad1) -> VDD
- J7 pad 2: ISINK_REF -> GND
- J8 pad 1: /DCC3_P_D_R_CC -> /DCC4_N_G_L_CS
- J8 pad 10: /DCC1_P_G_L_CS -> /DCC2_N_G_R_CC
- J8 pad 11: /DCC1_P_G_L_CC -> /DCC2_N_G_R_CS
- J8 pad 12: /DCC1_P_G_R_CS -> /DCC2_N_D_L_CC
- J8 pad 13: /DCC1_P_G_R_CC -> /DCC2_N_D_L_CS
- J8 pad 14: /DCC1_P_D_L_CS -> /DCC2_N_D_R_CC
- J8 pad 15: /DCC1_P_D_L_CC -> /DCC2_N_D_R_CS
- J8 pad 16: /DCC1_P_D_R_CS -> /DCC1_N_G_L_CC
- J8 pad 17: /DCC1_P_D_R_CC -> /DCC1_N_G_L_CS
- J8 pad 18: /DCC4_P_G_L_CS -> /DCC1_N_G_R_CC
- J8 pad 19: /DCC4_P_G_L_CC -> /DCC1_N_G_R_CS
- J8 pad 2: /DCC2_P_G_L_CS -> /DCC4_N_G_R_CC
- J8 pad 20: /DCC4_P_G_R_CS -> /DCC1_N_D_L_CC
- J8 pad 21: /DCC4_P_G_R_CC -> /DCC1_N_D_L_CS
- J8 pad 22: /DCC4_P_D_L_CS -> /DCC1_N_D_R_CC
- J8 pad 23: /DCC4_P_D_L_CC -> /DCC1_N_D_R_CS
- J8 pad 24: /DCC4_P_D_R_CS -> /DINV2_INP_L
- J8 pad 25: /DCC4_P_D_R_CC -> /DINV2_INN_L
- J8 pad 3: /DCC2_P_G_L_CC -> /DCC4_N_G_R_CS
- J8 pad 4: /DCC2_P_G_R_CS -> /DCC4_N_D_L_CC
- J8 pad 5: /DCC2_P_G_R_CC -> /DCC4_N_D_L_CS
- J8 pad 6: /DCC2_P_D_L_CS -> /DCC4_N_D_R_CC
- J8 pad 7: /DCC2_P_D_L_CC -> /DCC4_N_D_R_CS
- J8 pad 8: /DCC2_P_D_R_CS -> /DCC2_N_G_L_CC
- J8 pad 9: /DCC2_P_D_R_CC -> /DCC2_N_G_L_CS
- J9 pad 1: VDD -> /DINV2_OUT_L
- J9 pad 2: GND -> /DINV2_INP_R
- R1 pad 1: Net-(R1-Pad1) -> Net-(IC1-B1)
- R1 pad 2: Net-(C3-Pad1) -> Net-(D1-A)
- RV1 pad 2: Net-(R1-Pad1) -> Net-(J3-Pad1)
- U1 pad 4: LDO_PG_3.3V -> unconnected-(U1-PG-Pad4)
Routing:
- net GND: track 0.00 -> 443.3 mm, vias 0 -> 145
- net VDD: track 75.6 -> 346.5 mm, vias 0 -> 2
- net /CLK_SC: track 0.00 -> 61.9 mm
- net ISINK_REF: track 0.00 -> 59.0 mm
- net /DINV2_OUT_L: track 0.00 -> 51.4 mm
- net /DCC4_P_D_R_CC: track 0.00 -> 51.4 mm
- net /DCC4_P_D_L_CC: track 0.00 -> 50.9 mm
- net /DCC4_P_D_R_CS: track 0.00 -> 50.6 mm
- net /DINV2_INP_R: track 0.00 -> 49.6 mm
- net /DCC4_P_D_L_CS: track 0.00 -> 49.0 mm
- net /DINV2_INN_R: track 0.00 -> 48.6 mm
- net /EN: track 0.00 -> 48.3 mm
- net /DCC4_P_G_R_CC: track 0.00 -> 47.8 mm
- net /DINV2_OUT_R: track 0.00 -> 47.7 mm
- net /DCC4_P_G_R_CS: track 0.00 -> 47.0 mm
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- added copper zone on B.Cu, net GND
- added copper zone on F.Cu, net GND
Other:
- board outline added: 131.9 x 83.5 mm
- board text added: "+"
- board text added: "-"
- board text added: "1"
- board text added: "10"
- board text added: "100"
- board text added: "11"
- board text added: "12"
- board text added: "127mm"
- board text added: "13"
- board text added: "14"
- board text added: "15"
- board text added: "16"
- board text added: "17"
- board text added: "18"
- board text added: "19"
- board text added: "2"
- board text added: "20"
- board text added: "20250912"
- board text added: "21"
- board text added: "22"
- board text added: "23"
- board text added: "24"
- board text added: "25"
- board text added: "25k_POT_IREF"
- board text added: "25k_POT_VREF"
- board text added: "26"
- board text added: "27"
- board text added: "28"
- board text added: "29"
- board text added: "3"
- board text added: "30"
- board text added: "31"
- board text added: "32"
- board text added: "33"
- board text added: "34"
- board text added: "34.4mm"
- board text added: "35"
- board text added: "36"
- board text added: "37"
- board text added: "38"
- board text added: "39"
- board text added: "4"
- board text added: "40"
- board text added: "41"
- board text added: "42"
- board text added: "43"
- board text added: "44"
- board text added: "45"
- board text added: "46"
- board text added: "47"
- board text added: "48"
- board text added: "49"
- board text added: "5"
- board text added: "5.08mm (2 blocks on breadboard)"
- board text added: "50"
- board text added: "51"
- board text added: "52"
- board text added: "53"
- board text added: "54"
- board text added: "55"
- board text added: "56"
- board text added: "57"
- board text added: "58"
- board text added: "59"
- board text added: "6"
- board text added: "60"
- board text added: "61"
- board text added: "62"
- board text added: "63"
- board text added: "64"
- board text added: "65"
- board text added: "66"
- board text added: "67"
- board text added: "68"
- board text added: "69"
- board text added: "7"
- board text added: "7.62mm (3 blocks on breadboard)"
- board text added: "70"
- board text added: "71"
- board text added: "72"
- board text added: "73"
- board text added: "74"
- board text added: "75"
- board text added: "76"
- board text added: "77"
- board text added: "78"
- board text added: "78.5mm"
- board text added: "79"
- board text added: "8"
- board text added: "80"
- board text added: "81"
- board text added: "82"
- board text added: "83"
- board text added: "84"
- board text added: "85"
- board text added: "86"
- board text added: "87"
- board text added: "88"
- board text added: "89"
- board text added: "9"
- board text added: "90"
- board text added: "91"
- board text added: "92"
- board text added: "93"
- board text added: "94"
- board text added: "95"
- board text added: "96"
- board text added: "97"
- board text added: "98"
- board text added: "99"
- board text added: "AD8524"
- board text added: "AMP_BIN+"
- board text added: "AMP_BIN-"
- board text added: "AMP_BOUT"
- board text added: "CLK_MUX"
- board text added: "CLK_RPI"
- board text added: "DATA_MUX"
- board text added: "DATA_RPI_IN"
- board text added: "Daughter Card Plug-IN from here"
- board text added: "EN_MANUAL_IN"
- board text added: "EN_RPI_IN"
- board text added: "GND"
- board text added: "IREF_EN"
- board text added: "IREF_RES"
- board text added: "LDO"
- board text added: "LDO_3.3_OUT"
- board text added: "LDO_VIN"
- board text added: "LED_CLK_RPI"
- board text added: "LED_DATA_RPI"
- board text added: "LED_EN"
- board text added: "USB-C 5V IN"
- board text added: "USB_C_5V_OUT"
- board text added: "VDD_LDO_3.3"
- board text added: "VDD_RPI"
- board text added: "VREF"
- board text added: "VREF_EN"
- board text added: "VSS_RPI"
- board text added: "https://mosbius.org"

Commit message: 0919
Parts:
- added D4: LED_RED, MOSBius_V2_CHIP:LED_150120RS75000_WRE, F.Cu at (211.0, 112.1)
- added R6: 330, Resistor_SMD:R_0603_1608Metric, F.Cu at (206.3, 112.1)
Routing:
- net VDD: track 346.5 -> 350.9 mm
- net Net-(D4-A): track 0.00 -> 2.35 mm
Other:
- board text added: "POWER LED"
