File: Mother_Card/Mother_Card.kicad_sch (KiCad schematic)
At the start: 57 parts, among them IC1 AD8542ARMZ-REEL, IC2 SN74LVC1G3157DBVR, IC4 SN74LVC1G3157DBVR, J1 5-1746530-4, J11 Conn_01x25_Pin, J12 Conn_01x02_Pin, J13 PINHD_1x2_Male, J14 PINHD_1x2_Male, J14_GND1 Conn_01x03, J14_GND3 Conn_01x03, J15 USB4736, J16 Conn_02x02_Row_Letter_First, J2 PINHD_1x2_Male, J3 Conn_01x25_Pin, J4 Conn_01x25_Pin, J5 PINHD_1x2_Male, J7 PINHD_1x2_Male, J8 Conn_01x25_Pin, J9 PINHD_1x2_Male, U1 NCV8164ASN250T1G_LDO_2.5V

Commit message: update in 0912
Parts:
- removed C6: 1u, Capacitor_SMD:C_0603_1608Metric, symbol Symbols-Library:C_Small
- removed C7: 0.1u, Capacitor_SMD:C_0603_1608Metric, symbol Symbols-Library:C_Small
- removed J16: Conn_02x02_Row_Letter_First, Connector_PinHeader_2.54mm:PinHeader_2x02_P2.54mm_Vertical, symbol Connector_Generic:Conn_02x02_Row_Letter_First
- removed J_CLK_RPI: CLK_RPI, Connector_PinHeader_2.54mm:PinHeader_1x01_P2.54mm_Vertical, symbol Connector:Conn_01x01_Pin
- removed J_DATA_RPI: DATA_RPI, Connector_PinHeader_2.54mm:PinHeader_1x01_P2.54mm_Vertical, symbol Connector:Conn_01x01_Pin
- removed J_EN_3.3: EN_MANUAL(3.3V), Connector_PinHeader_2.54mm:PinHeader_1x01_P2.54mm_Vertical, symbol Connector:Conn_01x01_Pin
- removed J_EN_RPI: EN_RPI, Connector_PinHeader_2.54mm:PinHeader_1x01_P2.54mm_Vertical, symbol Connector:Conn_01x01_Pin
- added EN_TO_CHIP'1, VDD_GND_RPI1: PINHD_1x2_Male, Connector_PinHeader_2.54mm:PinHeader_1x02_P2.54mm_Vertical, symbol PCM_SL_Pin_Headers:PINHD_1x2_Male
- added J_CLK_RPI1: CLK_RPI, Connector_PinHeader_2.54mm:PinHeader_1x01_P2.54mm_Vertical, symbol Connector:Conn_01x01_Pin
- added J_DATA_RPI1: DATA_RPI, Connector_PinHeader_2.54mm:PinHeader_1x01_P2.54mm_Vertical, symbol Connector:Conn_01x01_Pin
- added OPAMP_1: Conn_01x03, Connector_PinHeader_2.54mm:PinHeader_1x03_P2.54mm_Vertical, symbol Symbols-Library:Conn_01x03
- IC2: renamed from IC1; footprint SOP65P490X110-8N -> MOSBius_V2_CHIP:AD8542
- renumbered C2 to C1, C4 to C10, C23 to C11, C5 to C12, C24 to C13, C25 to C14, C26 to C15, C18 to C16, C19 to C17, C20 to C18, C3 to C2, C1 to C3, C8 to C4, C11 to C5, C21 to C6, C13 to C7, C22 to C8, C17 to C9, D2 to D1, D1 to D2, IC2 to IC1, IC4 to IC3, J7 to J1, J15 to J10, J8 to J12, J12 to J13, J14_GND3 to J14_GND1, J14_GND1 to J14_GND2, J5 to J3, J1 to J5, J9 to J6, J13 to J7, J4 to J8, J3 to J9, J_VCM to J_VCM1, R3 to R1, R18 to R2, R1 to R3, R2 to R4, R4 to R5, RV2 to RV1, RV1 to RV2, Rd_2 to Rd_1
Connections:
- net CC_N_D_CS: now also J5.166; no longer J5.116
- net CC_N_G_CC: now also J5.172; no longer J5.122
- net CC_N_G_CS: now also J5.170; no longer J5.120
- net CC_P_D_CC: now also J5.174; no longer J5.124
- net CC_P_D_CS: now also J5.176; no longer J5.126
- net CC_P_G_CC: now also J5.178; no longer J5.128
- net CC_P_G_CS: now also J5.180; no longer J5.130
- net CLK: now also J5.5; no longer J5.55
- net CLK_SC: now also IC1.1 (B2); no longer IC1.3 (B1)
- net DATA_SBUS6: now also J5.7; no longer J5.57
- net DCC1_N_D_L_CC: now also J5.189; no longer J5.139
- net DCC1_N_D_L_CS: now also J5.191; no longer J5.141
- net DCC1_N_D_R_CC: now also J5.193; no longer J5.143
- net DCC1_N_D_R_CS: now also J5.195; no longer J5.145
- net DCC1_N_G_L_CC: now also J5.181; no longer J5.131
- net DCC1_N_G_L_CS: now also J5.183; no longer J5.133
- net DCC1_N_G_R_CC: now also J5.185; no longer J5.135
- net DCC1_N_G_R_CS: now also J5.187; no longer J5.137
- net DCC1_P_D_L_CC: now also J5.22; no longer J5.72
- net DCC1_P_D_L_CS: now also J5.24; no longer J5.74
- net DCC1_P_D_R_CC: now also J5.18; no longer J5.68
- net DCC1_P_D_R_CS: now also J5.20; no longer J5.70
- net DCC1_P_G_L_CC: now also J5.30; no longer J5.80
- net DCC1_P_G_L_CS: now also J5.32; no longer J5.82
- net DCC1_P_G_R_CC: now also J5.26; no longer J5.76
- net DCC1_P_G_R_CS: now also J5.28; no longer J5.78
- net DCC2_N_D_L_CC: now also J5.173; no longer J5.123
- net DCC2_N_D_L_CS: now also J5.175; no longer J5.125
- net DCC2_N_D_R_CC: now also J5.177; no longer J5.127
- net DCC2_N_D_R_CS: now also J5.179; no longer J5.129
- net DCC2_N_G_L_CC: now also J5.165; no longer J5.115
- net DCC2_N_G_L_CS: now also J5.167; no longer J5.117
- net DCC2_N_G_R_CC: now also J5.169; no longer J5.119
- net DCC2_N_G_R_CS: now also J5.171; no longer J5.121
- net DCC2_P_D_L_CC: now also J5.38; no longer J5.88
- net DCC2_P_D_L_CS: now also J5.40; no longer J5.90
- net DCC2_P_D_R_CC: now also J5.34; no longer J5.84
- net DCC2_P_D_R_CS: now also J5.36; no longer J5.86
- net DCC2_P_G_L_CC: now also J5.46; no longer J5.96
- net DCC2_P_G_L_CS: now also J5.48; no longer J5.98
- net DCC2_P_G_R_CC: now also J5.42; no longer J5.92
- net DCC2_P_G_R_CS: now also J5.44; no longer J5.94
- net DCC3_N_D_L_CC: now also J5.41; no longer J5.91
- net DCC3_N_D_L_CS: now also J5.43; no longer J5.93
- net DCC3_N_D_R_CC: now also J5.45; no longer J5.95
- net DCC3_N_D_R_CS: now also J5.47; no longer J5.97
- net DCC3_N_G_L_CC: now also J5.33; no longer J5.83
- net DCC3_N_G_L_CS: now also J5.35; no longer J5.85
- net DCC3_N_G_R_CC: now also J5.37; no longer J5.87
- net DCC3_N_G_R_CS: now also J5.39; no longer J5.89
- net DCC3_P_D_L_CC: now also J5.154; no longer J5.104
- net DCC3_P_D_L_CS: now also J5.156; no longer J5.106
- net DCC3_P_D_R_CC: now also J5.50; no longer J5.100
- net DCC3_P_D_R_CS: now also J5.152; no longer J5.102
- net DCC3_P_G_L_CC: now also J5.162; no longer J5.112
- net DCC3_P_G_L_CS: now also J5.164; no longer J5.114
- net DCC3_P_G_R_CC: now also J5.158; no longer J5.108
- net DCC3_P_G_R_CS: now also J5.160; no longer J5.110
- net DCC4_N_D_L_CC: now also J5.57; no longer J5.107
- net DCC4_N_D_L_CS: now also J5.59; no longer J5.109
- net DCC4_N_D_R_CC: now also J5.161; no longer J5.111
- net DCC4_N_D_R_CS: now also J5.163; no longer J5.113
- net DCC4_N_G_L_CC: now also J5.49; no longer J5.99
- net DCC4_N_G_L_CS: now also J5.51; no longer J5.101
- net DCC4_N_G_R_CC: now also J5.53; no longer J5.103
- net DCC4_N_G_R_CS: now also J5.55; no longer J5.105
- net DCC4_P_D_L_CC: now also J5.6; no longer J5.56
- net DCC4_P_D_L_CS: now also J5.8; no longer J5.58
- net DCC4_P_D_R_CC: now also J5.2; no longer J5.52
- net DCC4_P_D_R_CS: now also J5.4; no longer J5.54
- net DCC4_P_G_L_CC: now also J5.14; no longer J5.64
- net DCC4_P_G_L_CS: now also J5.16; no longer J5.66
- net DCC4_P_G_R_CC: now also J5.10; no longer J5.60
- net DCC4_P_G_R_CS: now also J5.12; no longer J5.62
- net DINV1_INN_L: now also J5.190; no longer J5.140
- net DINV1_INN_R: now also J5.184; no longer J5.134
- net DINV1_INP_L: now also J5.192; no longer J5.142
- net DINV1_INP_R: now also J5.186; no longer J5.136
- net DINV1_OUT_L: now also J5.188; no longer J5.138
- net DINV1_OUT_R: now also J5.182; no longer J5.132
- net DINV2_INN_L: now also J5.199; no longer J5.149
- net DINV2_INN_R: now also J5.196; no longer J5.146
- net DINV2_INP_L: now also J5.197; no longer J5.147
- net DINV2_INP_R: now also J5.198; no longer J5.148
- net DINV2_OUT_L: now also J5.200; no longer J5.150
- net DINV2_OUT_R: now also J5.194; no longer J5.144
- net EN: now also J5.3, EN_TO_CHIP'1.1, EN_TO_CHIP'1.2; no longer J5.53
- net GND: now also J11.1 (Pin_1), J11.2 (Pin_2), J5.100, J5.101, J5.102, J5.103, J5.104, J5.105, J5.106, J5.107, J5.108, J5.109, J5.110, J5.111, J5.112, J5.113, J5.114, J5.115, J5.116, J5.117, J5.118, J5.119, J5.120, J5.121, J5.122, J5.123, J5.124, J5.125, J5.126, J5.127, J5.128, J5.129, J5.130, J5.131, J5.132, J5.133, J5.134, J5.135, J5.136, J5.137, J5.138, J5.139, J5.140, J5.141, J5.142, J5.143, J5.144, J5.145, J5.146, J5.147, J5.148, J5.149, J5.150, J5.52, J5.54, J5.56, J5.58, J5.60, J5.61, J5.62, J5.63, J5.64, J5.65, J5.66, J5.67, J5.68, J5.69, J5.70, J5.71, J5.72, J5.73, J5.74, J5.75, J5.76, J5.77, J5.78, J5.79, J5.80, J5.81, J5.82, J5.83, J5.84, J5.85, J5.86, J5.87, J5.88, J5.89, J5.90, J5.91, J5.92, J5.93, J5.94, J5.95, J5.96, J5.97, J5.98, J5.99, VDD_GND_RPI1.2; no longer IC2.5 (+IN_B), IC2.6 (-IN_B), IC2.7 (OUT_B), J5.10, J5.11, J5.12, J5.13, J5.14, J5.15, J5.152, J5.154, J5.156, J5.158, J5.16, J5.160, J5.161, J5.162, J5.163, J5.164, J5.165, J5.166, J5.167, J5.168, J5.169, J5.17, J5.170, J5.171, J5.172, J5.173, J5.174, J5.175, J5.176, J5.177, J5.178, J5.179, J5.18, J5.180, J5.181, J5.182, J5.183, J5.184, J5.185, J5.186, J5.187, J5.188, J5.189, J5.19, J5.190, J5.191, J5.192, J5.193, J5.194, J5.195, J5.196, J5.197, J5.198, J5.199, J5.2, J5.20, J5.200, J5.21, J5.22, J5.23, J5.24, J5.25, J5.26, J5.27, J5.28, J5.29, J5.3, J5.30, J5.31, J5.32, J5.33, J5.34, J5.35, J5.36, J5.37, J5.38, J5.39, J5.4, J5.40, J5.41, J5.42, J5.43, J5.44, J5.45, J5.46, J5.47, J5.48, J5.49, J5.5, J5.50, J5.51, J5.6, J5.7, J5.8, J5.9, J5.MP1, J5.MP2
- net ISINK_REF: now also J5.168; no longer J5.118
- net OTA_N_INN: now also J5.29; no longer J5.79
- net OTA_N_INP: now also J5.27; no longer J5.77
- net OTA_N_OUT: now also J5.31; no longer J5.81
- net OTA_P_INN: now also J5.19; no longer J5.69
- net OTA_P_INP: now also J5.21; no longer J5.71
- net OTA_P_OUT: now also J5.23; no longer J5.73
- net SBUS1: now also J5.17; no longer J5.67
- net SBUS2: now also J5.15; no longer J5.65
- net SBUS3: now also J5.13; no longer J5.63
- net SBUS4: now also J5.11; no longer J5.61
- net SBUS5: now also J5.9; no longer J5.59
- net SBUS6: now also IC3.1 (B2); no longer IC3.3 (B1)
- net VDD: now also J5.25, VDD_GND_RPI1.1; no longer J5.75
- net at R5.1: now also IC3.3 (B1), J_DATA_RPI1.1 (Pin_1); no longer IC3.1 (B2)
- net at R1.1: now also IC1.3 (B1), J_CLK_RPI1.1 (Pin_1); no longer IC1.1 (B2)
- new net: IC2.7 (OUT_B), OPAMP_1.1 (Pin_1)
- new net: IC2.6 (-IN_B), OPAMP_1.2 (Pin_2)
- new net: IC2.5 (+IN_B), OPAMP_1.3 (Pin_3)
- no-connect marks 6 -> 4
Other:
- note added: "CLK input EN = 0 -> SW Matrix Program CLK from RPI EN = 1 -> External CLK used for SC CKT"
- note added: "DATA/SBUS6 input EN = 0 -> DATA from RPI EN = 1 -> SBUS6 on Chip"
- note added: "EN input (from RPI or Manually to 3.3V) EN = 0 -> Program from RPI EN = 1 -> Chip"
- note added: "EN_MAN_IN"
- note added: "EN_RPI_IN"
- note removed: "CLK input EN = 1 -> SW Matrix Program CLK from RPI EN = 0 -> External CLK used for SC CKT"
- note removed: "DATA/SBUS6 input EN = 1 -> DATA from RPI EN = 0 -> SBUS6 on Chip"
- note removed: "EN input (from RPI or Manually to 3.3V) EN = 1 -> Program from RPI EN = 0 -> Chip"
- moved on the sheet: C11, C13, C14, C15, C6, C8, J11, J12, J14, J7, J8, J9

Commit message: 0919
Parts:
- added D4: LED_RED, MOSBius_V2_CHIP:LED_150120RS75000_WRE, symbol Symbols-Library:LED
- added R6: 330, Resistor_SMD:R_0603_1608Metric, symbol Symbols-Library:R_1206
Connections:
- net GND: now also D4.1 (K)
- net VDD: now also R6.1
- new net: D4.2 (A), R6.2
