File: combined_board/combined_board.kicad_sch (KiCad schematic)
At the start: 57 parts, among them IC1 SN74LVC1G3157DBVR, IC2 AD8542ARMZ-REEL, IC3 SN74LVC1G3157DBVR, J1 PINHD_1x2_Male, J10 USB4736, J11 Conn_01x25_Pin, J12 Conn_01x25_Pin, J13 Conn_01x02_Pin, J14 PINHD_1x2_Male, J14_GND1 Conn_01x03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

Commit message: 0311_2026 XP update - mainly in RPI board
Parts:
- removed R2: 1k, Resistor_SMD:R_0603_1608Metric, symbol Symbols-Library:R_1206
- added J_VCM2: DIRECT_DATA_SBUS, Connector_PinHeader_2.54mm:PinHeader_1x01_P2.54mm_Vertical, symbol Connector:Conn_01x01_Pin
- added J_VCM3: DIRECT_CLK, Connector_PinHeader_2.54mm:PinHeader_1x01_P2.54mm_Vertical, symbol Connector:Conn_01x01_Pin
Connections:
- net CLK: now also J_VCM3.1 (Pin_1)
- net DATA_SBUS6: now also J_VCM2.1 (Pin_1)
Other:
- note added: "J_DATA_RPI, J_EN_RPI, J_CLK_RPI are headers connected to RPI J_EN_3.3 should connect to VDD (manually switch on EN) CLK_SC, SBUS6 pins are connected to breadboard DIRECT_DATA_SBUS is the header that direcly access to DATA_SBUS6 chip pin DIRECT_CLK is the header that direcly access to CLK chip pin"
- note added: "current measurement"
- note removed: "J_DATA_RPI, J_EN_RPI, J_CLK_RPI are headers connected to RPI J_EN_3.3 should connect to VDD (manually switch on EN) CLK_SC, SBUS6 pins are connected to breadboard"
- moved on the sheet: J3
